File: PianoTest/bus-pnp.kicad_sch (KiCad schematic)
At the start: 52 parts, among them J401 J_IN MAIN, J402 J_OUT MAIN, U401 74HC283, U402 74HC85, U403 74HC138, U404 SN74LVC2G17DBVR, U405 SN74LVC1G125DBVR, U406 SN74LVC1G332DBVR, U407 SN74LVC1G07DBVR, U408 25AA02E48T-I/SN

Commit message: Bus MIKILAB REV5.1: linea di coincidenza HIT# sul pin 28 del MAIN
Specifica: pin 28 (prima GND ridondante) = HIT#, open-drain attivo basso,
pull-up unico 4.7k sul master, impulso 100-200 ns per evento; logica di
coincidenza documentata (fronte marcato dal master, lettura dei latch).
PianoTest: HIT -> monostabile 74LVC1G123 (2k + 27 pF) -> 74LVC1G06 su
HIT#, passante J_IN -> J_OUT, ESD. ERC 0.
SchedaA133: J2 pin 28 -> PD4 (PD_EINT4), pull-up R336 4.7k, ESD su U307,
R337 0R DNP verso l'EXTINT del NEO-F10T. ERC 0, PDF rigenerato.
Documentazione bus della A133 e articolo (sezione bus e coincidenze)
aggiornati; corretta l'identita del primo piano (0).

Co-Authored-By: Claude Opus 5.5 (1M context) <noreply@anthropic.com>
Claude-Session: https://claude.ai/code/session_01J3krgWFTUEjwvCnwUp9cQn
Parts:
- added C415: 27pF C0G, Capacitor_SMD:C_0603_1608Metric, symbol Device:C
- added C416, C417: 100nF, Capacitor_SMD:C_0603_1608Metric, symbol Device:C
- added D420: TPD1E10B06, Diode_SMD:D_0402_1005Metric, symbol Device:D_TVS
- added R407: 2k, Resistor_SMD:R_0603_1608Metric, symbol Device:R
- added U409: SN74LVC1G123DCUR, Package_SO:VSSOP-8_2.3x2mm_P0.5mm, symbol PianoTest:74LVC1G123
- added U410: SN74LVC1G06DBVR, Package_TO_SOT_SMD:SOT-23-5, symbol PianoTest:74LVC1G06
Connections:
- net +3V3: now also C416.1, C417.1, R407.1, U409.3 (~{CLR}), U409.8 (VCC), U410.5 (VCC)
- net GND: now also C416.2, C417.2, D420.2 (A2), U409.1 (~{A}), U409.4 (GND), U410.3 (GND); no longer J401.28 (Pin_28), J402.28 (Pin_28)
- net ID_IN0: now also D415.1 (A1); no longer D414.1 (A1)
- net ID_IN1: now also D416.1 (A1); no longer D415.1 (A1)
- net ID_IN2: now also D417.1 (A1); no longer D416.1 (A1)
- net ID_OUT0: now also D418.1 (A1); no longer D417.1 (A1)
- net ID_OUT1: now also D419.1 (A1); no longer D418.1 (A1)
- net ID_OUT2: now also D420.1 (A1); no longer D419.1 (A1)
- new net BUS_HIT_N: D414.1 (A1), J401.28 (Pin_28), J402.28 (Pin_28), U410.4 (Y)
- new net HIT: U409.2 (B)
- new net HIT_PULSE: U409.5 (Q), U410.2 (A)
- new net MONO_C: C415.2, U409.6 (Cext)
- new net MONO_RC: C415.1, R407.2, U409.7 (Rext/Cext)
- no-connect marks 3 -> 4
Other:
- note added: "REV5.1: pin 28 = HIT# (open-drain, attivo basso, pull-up 4.7k sul master). HIT del comparatore -> monostabile 74LVC1G123 (2k + 27 pF, ~170-200 ns) -> 74LVC1G06 open-drain. Passante J_IN -> J_OUT."
