File: SchedaH616/progetto-kicad/cpu.kicad_sch (KiCad schematic)
At the start: 93 parts, among them J301 UART0 debug, SW301 RESET, SW302 FEL, U301 H616, U302 TPD4E05U06DQA, U303 TPD4E05U06DQA, U304 TPD4E05U06DQA, U305 TPD4E05U06DQA, U306 TPD4E05U06DQA, U307 TPD4E05U06DQA, U308 TCA6416APWR, Y301 24MHz

Commit message: SchedaH616: RK3568 + RK809-5 + TCS4525 + DDR4, placement 50x70
- SoC Allwinner H616 -> Rockchip RK3568 (FCBGA636L, LCSC C2938930): ball map dal pinout
  Rockchip V1.1, verificata sulla tabella 2-1 del datasheet V1.2 (636/636); footprint
  generato (gen_fp.py), confrontato con EasyEDA C2938930
- PMIC AXP313A -> RK809-5 (C2939628) come Rockchip AIoT REF V1.1 / ROCK 3A; TCS4525 per
  VDD_CPU su I2C0 (0x1C); BUCK4 su VDD_NPU (sull'RK809-5 parte spento: non puo' fare il 3.3 V)
- LPDDR4 -> DDR4 x16 K4AAG165WA-BCWE (C2920140) sul canale A, point-to-point, niente VTT,
  VPP da AP2112K-2.5, ZQ 240R, DDR_RZQ del SoC 120R (Hardware Design Guide)
- eMMC su EMMC 8 bit (VCCIO2 1.8 V), microSD su SDMMC0, AP6256 su SDMMC2 + UART8,
  RTL8211F su GMAC0 RGMII (22R TX al SoC e RX al PHY), console UART2_M0, USB-C su OTG0
- Recovery su SARADC_VIN0, reset sulla rete RESETn; TCA6416A tolto
- Bus MIKILAB: BUS_POWER su SPI3_M1, MAIN su SPI2_M1 (CS del DAC su cs-gpios)
- progetto rinominato SchedaRK3568, libreria di progetto Scheda; script portabili Linux/macOS
- ERC 0, parita' 0, DRC 0 (solo collegamenti da fare); placement 439/439

Co-Authored-By: Claude Opus 5.5 (1M context) <noreply@anthropic.com>
Parts:
- removed R340, R341, R342, R343, R344, R345, R346, R347: 10k, Resistor_SMD:R_0402_1005Metric, symbol Device:R
- removed U301: H616, H616:BGA-284_L14.0-W12.0-P0.65-TL, symbol H616:H616
- removed U308: TCA6416APWR, Package_SO:TSSOP-24_4.4x7.8mm_P0.65mm, symbol H616:TCA6416APWR
- added C336: 10uF, Capacitor_SMD:C_0603_1608Metric, symbol Device:C
- added C337, C339, C341, C343, C345, C352, C361: 1uF, Capacitor_SMD:C_0402_1005Metric, symbol Device:C
- added C338, C340, C342, C344, C346, C347, C348, C349, C350, C351, C353, C354, C355, C356, C357, C358, C359, C360: 100nF, Capacitor_SMD:C_0201_0603Metric, symbol Device:C
- added C362, C363: 1nF, Capacitor_SMD:C_0201_0603Metric, symbol Device:C
- added FB301, FB302: 120R@100MHz, Inductor_SMD:L_0603_1608Metric, symbol Device:FerriteBead
- added R335: 10k, Resistor_SMD:R_0402_1005Metric, symbol Device:R
- added U301: RK3568, Scheda:Rockchip_FCBGA-636_19x19mm_P0.65mm, symbol Scheda:RK3568
- C301, C302: value 12pF/50V -> 18pF/50V
- C303: value 220nF/16V -> 100nF
- C304: value 1nF/50V -> 1nF
- C305, C335: value 10uF/6.3V -> 4.7uF; footprint Capacitor_SMD:C_0603_1608Metric -> Capacitor_SMD:C_0402_1005Metric
- C306: value 2.2uF/6.3V -> 100nF; footprint Capacitor_SMD:C_0402_1005Metric -> Capacitor_SMD:C_0201_0603Metric
- C307, C311, C334: value 2.2uF/6.3V -> 4.7uF
- C308, C309: value 1uF -> 100nF; footprint Capacitor_SMD:C_0402_1005Metric -> Capacitor_SMD:C_0201_0603Metric
- C310: value 10uF/6.3V -> 100nF; footprint Capacitor_SMD:C_0603_1608Metric -> Capacitor_SMD:C_0201_0603Metric
- C312: value 2.2uF/6.3V -> 22uF; footprint Capacitor_SMD:C_0402_1005Metric -> Capacitor_SMD:C_0603_1608Metric
- C313, C314: value 1uF -> 22uF; footprint Capacitor_SMD:C_0402_1005Metric -> Capacitor_SMD:C_0603_1608Metric
- C315: value 1uF -> 22uF; footprint Capacitor_SMD:C_0402_1005Metric -> Capacitor_SMD:C_0603_1608Metric; now not fitted
- C316, C323, C328, C332, C333: value 0.1uF -> 100nF; footprint Capacitor_SMD:C_0402_1005Metric -> Capacitor_SMD:C_0201_0603Metric
- C317, C324: value 1uF -> 4.7uF
- C318, C319: value 0.1uF -> 1uF
- C320, C321, C325, C326: value 0.1uF -> 22uF; footprint Capacitor_SMD:C_0402_1005Metric -> Capacitor_SMD:C_0603_1608Metric
- C322, C327: value 0.1uF -> 10uF; footprint Capacitor_SMD:C_0402_1005Metric -> Capacitor_SMD:C_0603_1608Metric
- C329, C330: value 470nF/16V -> 22uF; footprint Capacitor_SMD:C_0402_1005Metric -> Capacitor_SMD:C_0603_1608Metric
- C331: value 1uF -> 10uF; footprint Capacitor_SMD:C_0402_1005Metric -> Capacitor_SMD:C_0603_1608Metric
- J301: value UART0 debug -> UART2 debug
- R301: value 0R -> 22R
- R302: value 10k -> 1M
- R304: value 240R 1% -> 10k
- R305, R310: value 33R -> 10k
- R306, R307, R308, R309: value 33R -> 2.2k
- R311, R312, R313: value 100R -> 10k
- R314, R315: value 100R -> 2.2R
- R316: value 100R -> 120R 1%
- R317, R318, R319, R320, R321: value 10k -> 33R
- R322: value 100k -> 33R
- R323: value 10k -> 100R
- R324, R325: value 4.7k -> 100R
- R326, R327, R328: value 2.2k -> 100R
- R329: value 2.2k -> 10k
- R334: value 10k -> 100k
- R336: value 0R -> 4.7k
- R337: value 150k 1% -> 4.7k
- R338: value 100R -> 2.2k
- R339: value 10k -> 2.2k
- SW302: value FEL -> RECOVERY
Connections:
- net 3V3_SYS is gone; now on net MAIN_SPI_ALERT_N: R336.2
- net IOX_INT_N is gone; now on net PWR_SPI_INA239B_CS: R330.2
- net IOX_RESET_N is gone; now on net PWR_SPI_DAC_CS: R331.2
- net PMU-SCK is gone; now on net MAIN_SPI_PREFIX_2: R328.2
- net PMU-SDA is gone; now on net PWR_SPI_INA239A_CS: R329.2
- net SOC_REXT is gone; now on net VCC_3V3: R337.1
- net SOC_VRA1 is gone; now on net VDD_NPU: C329.1
- net SOC_VRA2 is gone; now on net VDD_NPU: C330.1
- net SPI1_MISO is gone; now on net VCC3V3_PMU: R307.1, R310.1
- net SPI1_MOSI is gone; now on net VCC3V3_PMU: R306.1, R309.1
- net VDD-SYS is gone; now on net VDD_CPU: C310.1, C311.1, C312.1, C313.1
- net BT_HOST_WAKE: now also U301.AF23 (GPIO0_C1)
- net BT_REG_ON: now also U301.AA5 (GPIO3_D5)
- net BT_UART_CTS: now also U301.E25 (UART8_CTSn_M0/GPIO2_B2)
- net BT_UART_RTS: now also U301.D26 (UART8_RTSn_M0/GPIO2_B1)
- net BT_UART_RX: now also U301.E26 (UART8_RX_M0/GPIO2_C6)
- net BT_UART_TX: now also U301.F26 (UART8_TX_M0/GPIO2_C5)
- net BT_WAKE: now also U301.Y6 (GPIO3_D6)
- net DAC61402_FAULT: now also R335.2, U301.AG1 (GPIO3_B1); no longer R323.2
- net EMMC_CMD: now also U301.B22 (EMMC_CMD/GPIO1_C4)
- net EMMC_D0: now also U301.A24 (EMMC_D0/GPIO1_B4)
- net EMMC_D1: now also U301.C21 (EMMC_D1/GPIO1_B5)
- net EMMC_D2: now also U301.B24 (EMMC_D2/GPIO1_B6)
- net EMMC_D3: now also U301.D21 (EMMC_D3/GPIO1_B7)
- net EMMC_D4: now also U301.A25 (EMMC_D4/GPIO1_C0)
- net EMMC_D5: now also U301.E21 (EMMC_D5/GPIO1_C1)
- net EMMC_D6: now also U301.E22 (EMMC_D6/GPIO1_C2)
- net EMMC_D7: now also U301.B25 (EMMC_D7/GPIO1_C3)
- net EMMC_DS: now also U301.A26 (EMMC_DATA_STROBE/GPIO1_C6)
- net EMMC_RST: now also U301.F20 (EMMC_RSTn/GPIO1_C7)
- net GND_D: now also C329.2, C330.2, R316.2, R333.2, R334.2, C336.2, C337.2, C338.2, C339.2, C340.2, C341.2, C342.2, C343.2, C344.2, C345.2, C346.2, C347.2, C348.2, C349.2, C350.2, C351.2, C352.2, C353.2, C354.2, C355.2, C356.2, C357.2, C358.2, C359.2, C360.2, C361.2, C363.2, U301.A1 (VSS_1), U301.A10 (VSS_4), U301.A14 (VSS_5), U301.A18 (VSS_6), U301.A28 (VSS_7), U301.A3 (VSS_2), U301.A6 (VSS_3), U301.AA12 (AVSS_24), U301.AA14 (AVSS_25), U301.AA15 (AVSS_26), U301.AA17 (AVSS_27), U301.AA23 (VSS_135), U301.AA24 (AVSS_28), U301.AA26 (AVSS_29), U301.AA4 (VSS_133), U301.AA9 (VSS_134), U301.AB11 (AVSS_30), U301.AB12 (AVSS_31), U301.AB14 (AVSS_32), U301.AB15 (AVSS_33), U301.AB17 (AVSS_34), U301.AB2 (VSS_136), U301.AB24 (TVSS), U301.AB6 (VSS_137), U301.AC11 (AVSS_36), U301.AC12 (AVSS_37), U301.AC15 (AVSS_38), U301.AC18 (AVSS_39), U301.AC25 (AVSS_40), U301.AC26 (AVSS_41), U301.AC9 (AVSS_35), U301.AD26 (AVSS_42), U301.AD3 (VSS_138), U301.AE14 (AVSS_43), U301.AE17 (AVSS_44), U301.AE20 (AVSS_45), U301.AE21 (VSS_140), U301.AE27 (AVSS_46), U301.AE28 (AVSS_47), U301.AE6 (VSS_139), U301.AF11 (AVSS_49), U301.AF12 (AVSS_50), U301.AF14 (AVSS_51), U301.AF15 (AVSS_52), U301.AF17 (AVSS_53), U301.AF18 (AVSS_54), U301.AF20 (AVSS_55), U301.AF21 (AVSS_56), U301.AF26 (VSS_142), U301.AF3 (VSS_141), U301.AF9 (AVSS_48), U301.AG18 (AVSS_57), U301.AG5 (VSS_143), U301.AH1 (VSS_144), U301.AH18 (AVSS_58), U301.AH23 (AVSS_59), U301.AH28 (VSS_146), U301.AH8 (VSS_145), U301.B12 (VSS_10), U301.B16 (VSS_11), U301.B23 (VSS_12), U301.B26 (VSS_13), U301.B5 (VSS_8), U301.B9 (VSS_9), U301.C11 (VSS_18), U301.C12 (VSS_19), U301.C14 (VSS_20), U301.C15 (VSS_21), U301.C17 (VSS_22), U301.C18 (VSS_23), U301.C25 (VSS_24), U301.C3 (VSS_14), U301.C6 (VSS_15), U301.C8 (VSS_16), U301.C9 (VSS_17), U301.D11 (VSS_27), U301.D2 (VSS_25), U301.D28 (VSS_28), U301.D3 (VSS_26), U301.E3 (VSS_29), U301.E7 (VSS_30), U301.F1 (VSS_31), U301.F12 (VSS_34), U301.F14 (VSS_35), U301.F15 (VSS_36), U301.F17 (VSS_37), U301.F3 (VSS_32), U301.F9 (VSS_33), U301.G11 (VSS_42), U301.G12 (VSS_43), U301.G14 (VSS_44), U301.G15 (VSS_45), U301.G17 (VSS_46), U301.G18 (VSS_47), U301.G24 (VSS_48), U301.G5 (VSS_38), U301.G6 (VSS_39), U301.G8 (VSS_40), U301.G9 (VSS_41), U301.H2 (VSS_49), U301.H3 (VSS_50), U301.H6 (VSS_51), U301.J17 (VSS_54), U301.J18 (VSS_55), U301.J20 (VSS_56), U301.J22 (VSS_57), U301.J26 (VSS_58), U301.J27 (AVSS_1), U301.J3 (VSS_52), U301.J5 (VSS_53), U301.J8 (DDR_AVSS), U301.K1 (VSS_59), U301.K11 (VSS_60), U301.K12 (VSS_61), U301.K13 (VSS_62), U301.K14 (VSS_63), U301.K19 (VSS_64), U301.L11 (VSS_68), U301.L13 (VSS_69), U301.L14 (VSS_70), U301.L19 (VSS_71), U301.L20 (VSS_72), U301.L21 (VSS_73), U301.L24 (AVSS_2), U301.L26 (AVSS_3), U301.L3 (VSS_65), U301.L5 (VSS_66), U301.L8 (VSS_67), U301.M11 (VSS_78), U301.M13 (VSS_79), U301.M14 (VSS_80), U301.M16 (VSS_81), U301.M18 (VSS_82), U301.M2 (VSS_74), U301.M20 (EDP_TX_AVDD_0V9), U301.M21 (AVSS_4), U301.M22 (EDP_TX_AVDD_1V8), U301.M26 (AVSS_5), U301.M3 (VSS_75), U301.M6 (VSS_76), U301.M8 (VSS_77), U301.N1 (VSS_83), U301.N11 (SYSPLL_AVSS), U301.N12 (VSS_84), U301.N14 (VSS_85), U301.N15 (VSS_86), U301.N17 (VSS_87), U301.N18 (VSS_88), U301.N28 (AVSS_6), U301.P10 (USB2_AVDD_3V3), U301.P12 (VSS_91), U301.P14 (VSS_92), U301.P15 (VSS_93), U301.P17 (VSS_94), U301.P21 (AVSS_7), U301.P26 (AVSS_8), U301.P3 (VSS_89), U301.P6 (VSS_90), U301.P9 (USB2_AVDD_1V8), U301.R10 (VSS_97), U301.R11 (VSS_98), U301.R14 (VSS_99), U301.R15 (VSS_100), U301.R17 (VSS_101), U301.R18 (VSS_102), U301.R19 (VSS_103), U301.R20 (MULTI_PHY_AVDD_0V9_1), U301.R21 (MULTI_PHY_AVDD_0V9_2), U301.R22 (MULTI_PHY_AVDD_1V8), U301.R23 (AVSS_9), U301.R26 (AVSS_10), U301.R3 (VSS_95), U301.R6 (VSS_96), U301.R8 (USB2_AVDD_0V9), U301.T10 (VSS_104), U301.T11 (VSS_105), U301.T14 (VSS_106), U301.T15 (VSS_107), U301.T17 (VSS_108), U301.T18 (VSS_109), U301.T19 (VSS_110), U301.U1 (VSS_111), U301.U10 (VSS_115), U301.U14 (VSS_116), U301.U15 (VSS_117), U301.U16 (VSS_118), U301.U17 (VSS_119), U301.U18 (VSS_120), U301.U20 (PCIE30_AVDD_0V9_2), U301.U21 (PCIE30_AVDD_0V9_1), U301.U22 (PCIE30_AVDD_1V8), U301.U23 (AVSS_11), U301.U26 (AVSS_12), U301.U6 (VSS_112), U301.U7 (VSS_113), U301.U8 (VSS_114), U301.V13 (VSS_124), U301.V14 (AVSS_13), U301.V15 (AVSS_14), U301.V16 (AVSS_15), U301.V17 (HDMI_TX_AVDD_0V9_1), U301.V18 (HDMI_TX_AVDD_0V9_2), U301.V20 (PMUPLL_AVSS), U301.V22 (AVSS_16), U301.V23 (AVSS_17), U301.V26 (AVSS_18), U301.V3 (VSS_121), U301.V8 (VSS_122), U301.V9 (VSS_123), U301.W10 (VSS_125), U301.W11 (VSS_126), U301.W12 (VSS_127), U301.W13 (VSS_128), U301.W14 (MIPI_CSI_RX_AVDD_0V9), U301.W15 (MIPI_DSI_TX1_AVDD_0V9), U301.W16 (MIPI_DSI_TX0), U301.W17 (AVSS_19), U301.W18 (HDMI_TX_AVDD_1V8), U301.Y11 (VSS_131), U301.Y12 (VSS_132), U301.Y14 (MIPI_CSI_RX_AVDD_1V8), U301.Y15 (MIPI_DSI_TX1_AVDD_1V8), U301.Y17 (MIPI_DSI_TX0), U301.Y18 (AVSS_20), U301.Y23 (AVSS_21), U301.Y24 (AVSS_22), U301.Y26 (AVSS_23), U301.Y8 (VSS_129), U301.Y9 (VSS_130); no longer R303.2, R304.2, R321.2, R322.2
- net GNSS_EXTINT: now also U301.AG3 (GPIO3_A6)
- net GNSS_PPS: now also U301.AH3 (GPIO3_A5)
- net MAIN_HIT_N: now also R337.2, U301.AF4 (GPIO3_A4); no longer R325.2
- net MAIN_I2C_SCL: now also R338.2, U301.AE2 (I2C3_SCL_M1/GPIO3_B5); no longer R326.2
- net MAIN_I2C_SDA: now also R339.2, U301.AE3 (I2C3_SDA_M1/GPIO3_B6); no longer R327.2
- net MAIN_SPI_ADDR_0: now also R323.2; no longer R311.2
- net MAIN_SPI_ADDR_1: now also R324.2; no longer R312.2
- net MAIN_SPI_ADDR_2: now also R325.2; no longer R313.2
- net MAIN_SPI_ALERT_N: now also U301.AG4 (GPIO3_A3); no longer R324.2
- net MAIN_SPI_CS_MASTER: now also R332.2, U301.AF6 (SPI2_CS0_M1/GPIO2_D5); no longer R320.2
- net MAIN_SPI_MISO: now also R322.2; no longer R310.2
- net MAIN_SPI_MOSI: now also R321.2; no longer R309.2
- net MAIN_SPI_PREFIX_0: now also R326.2; no longer R314.2
- net MAIN_SPI_PREFIX_1: now also R327.2; no longer R315.2
- net MAIN_SPI_PREFIX_2: no longer R316.2
- net MAIN_SPI_SCLK: now also R320.2; no longer R308.2
- net PD_INT_N: now also R311.2, U301.AC22 (GPIO0_B5); no longer R332.2
- net PHY_EE_CS_N: now also U301.AF5 (SPI2_CS1_M1/GPIO2_D4)
- net PHY_INT_N: now also U301.AA3 (GPIO4_A0)
- net PHY_MDC: now also U301.H24 (GMAC0_MDC/GPIO2_C3)
- net PHY_MDIO: now also U301.H23 (GMAC0_MDIO/GPIO2_C4)
- net PHY_RST_N: now also U301.Y5 (GPIO3_D7)
- net PWR_SPI_DAC_CS: now also U301.AH7 (GPIO4_C4); no longer R319.2
- net PWR_SPI_INA239A_CS: now also U301.AE8 (SPI3_CS0_M1/GPIO4_C6); no longer R317.2
- net PWR_SPI_INA239B_CS: now also U301.AH6 (SPI3_CS1_M1/GPIO4_D1); no longer R318.2
- net PWR_SPI_MISO: now also R319.2; no longer R307.2
- net PWR_SPI_MOSI: now also R318.2; no longer R306.2
- net PWR_SPI_SCLK: now also R317.2; no longer R305.2
- net PWR_SRC_ST: now also R313.2, U301.AH26 (GPIO0_B7); no longer R334.2
- net RGMII_CLKIN: now also U301.F25 (GMAC0_MCLKINOUT/GPIO2_C2)
- net RGMII_RXCK: now also U301.B28 (GMAC0_RXCLK/GPIO2_A5)
- net RGMII_RXCTL: now also U301.F24 (GMAC0_RXDV_CRS/GPIO2_C0)
- net RGMII_RXD0: now also U301.F27 (GMAC0_RXD0/GPIO2_B6)
- net RGMII_RXD1: now also U301.H25 (GMAC0_RXD1/GPIO2_B7)
- net RGMII_RXD2: now also U301.E27 (GMAC0_RXD2/GPIO2_A3)
- net RGMII_RXD3: now also U301.E28 (GMAC0_RXD3/GPIO2_A4)
- net RGMII_TXCK: now also U301.D27 (GMAC0_TXCLK/GPIO2_B0)
- net RGMII_TXCTL: now also U301.G28 (GMAC0_TXEN/GPIO2_B5)
- net RGMII_TXD0: now also U301.F28 (GMAC0_TXD0/GPIO2_B3)
- net RGMII_TXD1: now also U301.G27 (GMAC0_TXD1/GPIO2_B4)
- net RGMII_TXD2: now also U301.C27 (GMAC0_TXD2/GPIO2_A6)
- net RGMII_TXD3: now also U301.C28 (GMAC0_TXD3/GPIO2_A7)
- net SD_CMD: now also U301.H27 (SDMMC0_CMD/GPIO2_A1)
- net SD_D0: now also U301.J25 (SDMMC0_D0/GPIO1_D5)
- net SD_D1: now also U301.J24 (SDMMC0_D1/GPIO1_D6)
- net SD_D2: now also U301.H26 (SDMMC0_D2/GPIO1_D7)
- net SD_D3: now also U301.J23 (SDMMC0_D3/GPIO2_A0)
- net SD_DET: now also U301.Y22 (SDMMC0_DET/GPIO0_A4)
- net SOC_ADDR_0: now also R323.1, U301.AG6 (GPIO2_D0); no longer R311.1
- net SOC_ADDR_1: now also R324.1, U301.AD7 (GPIO2_D1); no longer R312.1
- net SOC_ADDR_2: now also R325.1, U301.AC8 (GPIO2_D2); no longer R313.1
- net SOC_PREFIX_0: now also R326.1, U301.AC7 (GPIO2_D3); no longer R314.1
- net SOC_PREFIX_1: now also R327.1, U301.AB8 (GPIO3_A1); no longer R315.1
- net SOC_PREFIX_2: now also R328.1, U301.AE5 (GPIO3_A2); no longer R316.1
- net USB0_DM: now also R315.1
- net USB0_DP: now also R314.1
- net USB1_DM: now also U301.P25 (USB3_HOST1_DM)
- net USB1_DP: now also U301.P24 (USB3_HOST1_DP)
- net USB1_OC_N: now also R312.2, U301.AA20 (GPIO0_B6); no longer R333.2
- net USB1_VBUS_EN: now also U301.AE24 (GPIO0_A6)
- net VBIAS_ENABLE: now also R334.1, U301.AG2 (GPIO3_B0); no longer R322.1
- net VBUS_SRC_EN: now also U301.AF25 (GPIO0_A5)
- net VREF_ENABLE: now also R333.1, U301.AH2 (GPIO3_A7); no longer R321.1
- net WL_HOST_WAKE: now also U301.AD22 (GPIO0_C0)
- net WL_REG_ON: now also U301.AA1 (GPIO3_D4)
- net WL_SDIO_CMD: now also U301.Y7 (SDMMC2_CMD_M0/GPIO3_D2)
- net WL_SDIO_D0: now also U301.AC5 (SDMMC2_D0_M0/GPIO3_C6)
- net WL_SDIO_D1: now also U301.AA6 (SDMMC2_D1_M0/GPIO3_C7)
- net WL_SDIO_D2: now also U301.AB5 (SDMMC2_D2_M0/GPIO3_D0)
- net WL_SDIO_D3: now also U301.AB1 (SDMMC2_D3_M0/GPIO3_D1)
- net AP-RESET renamed VCC_3V3
- net VCC_3V3: now also C309.1, R329.1, R330.1, R331.1, R332.1, R336.1, R339.1, C354.1, C355.1, C356.1, C357.1, C358.1, C359.1, C360.1, C361.1, R335.1, U301.J21 (VCCIO4), U301.M23 (USB3_AVDD_3V3), U301.R9 (VCCIO6_1), U301.U9 (VCCIO6_2), U301.V10 (VCCIO5_1), U301.V11 (VCCIO5_2), U301.V12 (VCCIO7)
- net DCXO_XIN renamed XTAL24_X1
- net XTAL24_X1: now also R301.2
- net DCXO_XOUT renamed XOUT24M
- net XOUT24M: now also R302.2, U301.AF27 (XOUT24M)
- net DCXO_XOUT_R renamed XIN24M
- net XIN24M: now also R302.1, U301.AF28 (XIN24M); no longer R301.2
- net SOC_AC_VRA1 renamed VDD_NPU
- net VDD_NPU: now also C328.1, U301.M19 (VDD_NPU_1), U301.N19 (VDD_NPU_2), U301.P18 (VDD_NPU_3), U301.P19 (VDD_NPU_4), U301.P20 (VDD_NPU_5)
- removed net SOC_AGND: C329.2, C330.2, R303.1, R337.2
- net SOC_DXLDO renamed RESETn
- net RESETn: now also R303.2, SW301.1, U301.AH27 (nPOR_u)
- net SOC_FEL renamed SARADC_VIN0
- net SARADC_VIN0: now also C304.1, R305.2, U301.B27 (SARADC_VIN0); no longer R302.2
- removed net SOC_RESET: C304.1, R338.2, R339.2, SW301.1
- net SOC_SZQ renamed VCC3V3_PMU
- net VCC3V3_PMU: now also R308.1, R311.1, R312.1, R313.1, C349.1, C350.1, U301.W19 (PMUIO2), U301.Y20 (PMUIO1)
- net SPI1_CLK renamed VCCA_1V8
- net VCCA_1V8: now also C345.1, C346.1, C347.1, C348.1, FB302.1, U301.H20 (OTP_VCC18), U301.H22 (SARADC_AVDD_1V8), U301.N10 (SYSPLL_AVDD_1V8); no longer R308.1
- net UART0_RX renamed UART2_RX
- net UART2_RX: now also U301.AC20 (UART2_RX_M0/GPIO0_D0)
- net UART0_TX renamed UART2_TX
- net UART2_TX: now also U301.AH24 (UART2_TX_M0/GPIO0_D1)
- removed net VCC-1V8: C317.1, C318.1, C319.1, C320.1, C321.1, C322.1, C332.1, C334.1, C335.1, R328.1, R329.1, R331.1, R339.1
- removed net VCC-1V8-EMMC: C323.1, R330.1, R332.1, R333.1
- net VCC-DRAM renamed VDD_CPU
- net VDD_CPU: now also U301.J15 (VDD_CPU_1), U301.K15 (VDD_CPU_2), U301.K16 (VDD_CPU_3), U301.K17 (VDD_CPU_4), U301.K18 (VDD_CPU_5), U301.L15 (VDD_CPU_6), U301.L16 (VDD_CPU_7), U301.L17 (VDD_CPU_8), U301.L18 (VDD_CPU_9), U301.M17 (VDD_CPU_10); no longer C316.1
- removed net VCC-IO: C324.1, C325.1, C326.1, C327.1, C328.1, C333.1, R302.1, R317.1, R318.1, R319.1, R320.1, R323.1, R324.1, R325.1, R326.1, R327.1, R334.1, R336.1
- removed net VDD-CPU: C305.1, C306.1, C307.1, C308.1, C309.1
- new net CLK32K: U301.AD23 (CLK32K_IN/GPIO0_B0)
- new net DDR_A0: U301.B6 (AC0/DDR4_A0)
- new net DDR_A1: U301.F5 (AC1/DDR4_A1)
- new net DDR_A10: U301.D6 (AC10/DDR4_A10)
- new net DDR_A11: U301.C2 (AC11/DDR4_A11)
- new net DDR_A12: U301.C4 (AC12/DDR4_A12)
- new net DDR_A13: U301.B8 (AC13/DDR4_A13)
- new net DDR_A14_WE_N: U301.C5 (AC14/DDR4_A14_WEn)
- new net DDR_A15_CAS_N: U301.E4 (AC15/DDR4_A15_CASn)
- new net DDR_A16_RAS_N: U301.D5 (AC16/DDR4_A16_RASn)
- new net DDR_A2: U301.B1 (AC2/DDR4_A2)
- new net DDR_A3: U301.F4 (AC3/DDR4_A3)
- new net DDR_A4: U301.D9 (AC4/DDR4_A4)
- new net DDR_A5: U301.B7 (AC5/DDR4_A5)
- new net DDR_A6: U301.A7 (AC6/DDR4_A6)
- new net DDR_A7: U301.A8 (AC7/DDR4_A7)
- new net DDR_A8: U301.C1 (AC8/DDR4_A8)
- new net DDR_A9: U301.A5 (AC9/DDR4_A9)
- new net DDR_ACT_N: U301.E6 (AC17/DDR4_ACTn)
- new net DDR_BA0: U301.E11 (AC18/DDR4_BA0)
- new net DDR_BA1: U301.E9 (AC19/DDR4_BA1)
- new net DDR_BG0: U301.F8 (AC20/DDR4_BG0)
- new net DDR_CKE: U301.B3 (AC22/DDR4_CKE)
- new net DDR_CK_N: U301.A4 (AC24/DDR4_CLKN)
- new net DDR_CK_P: U301.B4 (AC23/DDR4_CLKP)
- new net DDR_CS_N: U301.A2 (AC25/DDR4_CS0n)
- new net DDR_DML: U301.H5 (DDR_DM0_A/DDR4_DML_A)
- new net DDR_DMU: U301.J4 (DDR_DM1_A/DDR4_DMU_A)
- new net DDR_DQL0: U301.F2 (DDR_DQ0_A/DDR4_DQL0_A)
- new net DDR_DQL1: U301.H4 (DDR_DQ7_A/DDR4_DQL1_A)
- new net DDR_DQL2: U301.E1 (DDR_DQ1_A/DDR4_DQL2_A)
- new net DDR_DQL3: U301.H1 (DDR_DQ6_A/DDR4_DQL3_A)
- new net DDR_DQL4: U301.E2 (DDR_DQ2_A/DDR4_DQL4_A)
- new net DDR_DQL5: U301.J2 (DDR_DQ5_A/DDR4_DQL5_A)
- new net DDR_DQL6: U301.D1 (DDR_DQ3_A/DDR4_DQL6_A)
- new net DDR_DQL7: U301.J1 (DDR_DQ4_A/DDR4_DQL7_A)
- new net DDR_DQSL_N: U301.G2 (DDR_DQS0N_A/DDR4_DQSL_N_A)
- new net DDR_DQSL_P: U301.G1 (DDR_DQS0P_A/DDR4_DQSL_P_A)
- new net DDR_DQSU_N: U301.L1 (DDR_DQS1N_A/DDR4_DQSU_N_A)
- new net DDR_DQSU_P: U301.L2 (DDR_DQS1P_A/DDR4_DQSU_P_A)
- new net DDR_DQU0: U301.L4 (DDR_DQ15_A/DDR4_DQU0_A)
- new net DDR_DQU1: U301.N2 (DDR_DQ9_A/DDR4_DQU1_A)
- new net DDR_DQU2: U301.K2 (DDR_DQ12_A/DDR4_DQU2_A)
- new net DDR_DQU3: U301.M1 (DDR_DQ8_A/DDR4_DQU3_A)
- new net DDR_DQU4: U301.J6 (DDR_DQ13_A/DDR4_DQU4_A)
- new net DDR_DQU5: U301.L6 (DDR_DQ11_A/DDR4_DQU5_A)
- new net DDR_DQU6: U301.J7 (DDR_DQ14_A/DDR4_DQU6_A)
- new net DDR_DQU7: U301.L7 (DDR_DQ10_A/DDR4_DQU7_A)
- new net DDR_ODT: U301.E8 (AC27/DDR4_ODT0)
- new net DDR_RESET_N: U301.F11 (AC29/DDR4_RESETn)
- new net DDR_VREFOUT: C362.1, C363.1, U301.P8 (DDR_VREFOUT)
- new net EMMC_CLK_S: U301.A23 (EMMC_CLKOUT/GPIO1_C5)
- new net FLASH_VOL_SEL: R304.2, U301.AG25 (FLASH_VOL_SEL/GPIO0_A7)
- new net GNSS_UART_RX: U301.AD2 (UART3_RX_M1/GPIO3_C0)
- new net GNSS_UART_TX: U301.AD4 (UART3_TX_M1/GPIO3_B7)
- new net I2C0_SCL: R306.2, U301.AF24 (I2C0_SCL/GPIO0_B1)
- new net I2C0_SDA: R307.2, U301.AB21 (I2C0_SDA/GPIO0_B2)
- new net I2C1_SCL: R308.2, U301.AG24 (I2C1_SCL/GPIO0_B3)
- new net I2C1_SDA: R309.2, U301.AB20 (I2C1_SDA/GPIO0_B4)
- new net OTG_VBUSDET: U301.M24 (USB3_OTG0_VBUSDET)
- new net PMIC_INT_L: R310.2, U301.AA22 (GPIO0_A3)
- new net PMIC_SLEEP_H: U301.AG28 (PMIC_SLEEP/GPIO0_A2)
- new net SD_CLK_S: U301.H28 (SDMMC0_CLK/GPIO2_A2)
- new net SOC_DDR_RZQ: R316.1, U301.H7 (DDR_RZQ)
- new net SPI2_CLK: R320.1, U301.AH4 (SPI2_CLK_M1/GPIO3_A0)
- new net SPI2_MISO: R322.1, U301.AH5 (SPI2_MISO_M1/GPIO2_D7)
- new net SPI2_MOSI: R321.1, U301.AD6 (SPI2_MOSI_M1/GPIO2_D6)
- new net SPI3_CLK: R317.1, U301.AF8 (SPI3_CLK_M1/GPIO4_C2)
- new net SPI3_MISO: R319.1, U301.AD8 (SPI3_MISO_M1/GPIO4_C5)
- new net SPI3_MOSI: R318.1, U301.AA11 (SPI3_MOSI_M1/GPIO4_C3)
- new net TSADC_SHUT: R303.1, U301.AG26 (TSADC_SHUT_M0/GPIO0_A1)
- new net USB_AVDD_0V9: C305.1, C306.1, FB301.2, U301.P22 (USB3_AVDD_0V9)
- new net USB_AVDD_1V8: C307.1, C308.1, FB302.2, U301.P23 (USB3_AVDD_1V8)
- new net USB_OTG0_DM_S: R315.2, U301.P28 (USB3_OTG0_DM)
- new net USB_OTG0_DP_S: R314.2, U301.P27 (USB3_OTG0_DP)
- new net VCC1V8_EMMC: C351.1, C352.1, U301.H18 (VCCIO2)
- new net VCCA1V8_PMU: C341.1, C342.1, U301.Y21 (PMUPLL_AVDD_1V8)
- new net VCCIO_SD: C353.1, U301.L22 (VCCIO3)
- new net VCC_DDR: C332.1, C333.1, C334.1, C335.1, C336.1, C362.2, U301.H11 (DDRPHY_VDDQ_2), U301.H12 (DDRPHY_VDDQ_3), U301.H14 (DDRPHY_VDDQ_4), U301.H15 (DDRPHY_VDDQ_5), U301.H9 (DDRPHY_VDDQ_1), U301.J11 (DDRPHY_VDDQL_1), U301.J12 (DDRPHY_VDDQL_2), U301.J14 (DDRPHY_VDDQL_3), U301.J9 (DDRPHY_VDDQ_6), U301.K10 (DDRPHY_VDDQL_4), U301.L10 (DDRPHY_VDDQL_5), U301.L9 (DDRPHY_VDDQ_7), U301.M10 (DDRPHY_VDDQL_6), U301.M9 (DDRPHY_VDDQ_8)
- new net VDDA0V9_PMU: C337.1, C338.1, C339.1, C340.1, U301.V19 (PMU_VDD_LOGIC_0V9), U301.V21 (PMUPLL_AVDD_0V9)
- new net VDDA_0V9: C343.1, C344.1, FB301.1, U301.P11 (SYSPLL_AVDD_0V9)
- new net VDD_CPU_COM: U301.M15 (VDD_CPU_COM)
- new net VDD_GPU: C323.1, C324.1, C325.1, C326.1, C327.1, U301.R13 (VDD_GPU_1), U301.T13 (VDD_GPU_2), U301.U11 (VDD_GPU_3), U301.U12 (VDD_GPU_4), U301.U13 (VDD_GPU_5)
- new net VDD_LOGIC: C316.1, C317.1, C318.1, C319.1, C320.1, C321.1, C322.1, U301.L12 (VDD_LOGIC_1), U301.M12 (VDD_LOGIC_2), U301.N13 (VDD_LOGIC_3), U301.N16 (VDD_LOGIC_4), U301.P13 (VDD_LOGIC_5), U301.P16 (VDD_LOGIC_6), U301.R12 (VDD_LOGIC_7), U301.R16 (VDD_LOGIC_8), U301.T12 (VDD_LOGIC_9), U301.T16 (VDD_LOGIC_10)
- new net WL_SDIO_CLK_S: U301.AC1 (SDMMC2_CLK_M0/GPIO3_D3)
- no-connect marks 72 -> 212
Other:
- note added: "24 MHz (Hardware Design Guide RK3568 fig. 2-1 / reference AIoT): 22R serie su XOUT24M, 1M tra XIN e XOUT, 18 pF per lato (da adattare al CL del quarzo, tolleranza 20 ppm)."
- note added: "BUS_POWER su SPI3_M1 (VCCIO7): CLK GPIO4_C2, MOSI GPIO4_C3, MISO GPIO4_C5, CS0 INA239A GPIO4_C6, CS1 INA239B GPIO4_D1; CS del DAC su GPIO4_C4 con cs-gpios (SPI3 ha solo due CS hardware)."
- note added: "C315 DNP: 22 uF di riserva su VDD_CPU (Hardware Design Guide). VCCIO4 ha due 100 nF (RGMII), VCCIO5/VCCIO6 due sfere ciascuno."
- note added: "CPU: Rockchip RK3568 (FCBGA636L 19x19 mm, passo 0.65 mm, LCSC C2938930). Ball map: Rockchip RK3568 PinOut V1.1, verificata sulla tabella 2-1 del datasheet V1.2 (636/636). Serie 3xx."
- note added: "DDR4 a 16 bit sul canale A del PHY (DQ0-15_A, nomi DDR4_DQL/DQU_A del pinout Rockchip); canale B, ECC, CS1n, ODT1, BG1 non usati. Mappa completa in docs/pinmap-rk3568.md."
- note added: "DDR_RZQ (H7): 120R 1% a GND per DDR4 (Hardware Design Guide 2.1.7.2; l'appunto diceva 240R, che vale per lo ZQ della DDR4). DDR_VREFOUT (P8): 1 nF a VCC_DDR e 1 nF a GND vicino al SoC."
- note added: "Disaccoppiamento secondo il reference Rockchip RK3568 AIoT V1.1: 100 nF/1 nF in 0201 e 4.7 uF/1 uF in 0402 sotto il package, 22 uF/10 uF 0603 vicino."
- note added: "Domini IO: PMUIO1/PMUIO2 = VCC3V3_PMU (3.3 V), VCCIO2 = VCC1V8_EMMC (1.8 V, FLASH_VOL_SEL alto), VCCIO3 = VCCIO_SD, VCCIO4-7 = VCC_3V3 (3.3 V), VCCIO1 non usato (flottante, come da Rockchip)."
- note added: "I2C del bus su I2C3_M1 (GPIO3_B5/B6). ADDR/PREFIX con 100R serie. Linee lente (VREF/VBIAS_ENABLE, FAULT, ALERT#, HIT#, PPS, EXTINT) su GPIO diretti: niente TCA6416A."
- note added: "I2C0 (GPIO0_B1/B2, PMUIO2): RK809-5 0x20 e TCS4525 0x1C, pull-up 2.2k a VCC3V3_PMU. I2C1 (GPIO0_B3/B4): FUSB302B 0x22, 2.2k a VCC3V3_PMU."
- note added: "Il tasto RESET tira giu' RESETn: l'RK809-5 rifa' la sequenza di accensione (Hardware Design Guide, par. Reset). FLASH_VOL_SEL (GPIO0_A7) 10k a VCC3V3_PMU: VCCIO2 a 1.8 V."
- note added: "J301 console UART2_M0 (GPIO0_D1 TX, GPIO0_D0 RX, PMUIO2 3.3 V): 1 = TX del SoC, 2 = RX del SoC, 3 = GND. 1500000 baud (default Rockchip)."
- note added: "Livelli di riposo: CS e CS_MASTER alti (10k), VREF_ENABLE basso (10k a GND), VBIAS_ENABLE basso (100k a GND), ALERT# e HIT# 4.7k, I2C del bus 2.2k, FAULT 10k (tutti a VCC_3V3)."
- note added: "MAIN su SPI2_M1 (VCCIO5): CLK GPIO3_A0, MOSI GPIO2_D6, MISO GPIO2_D7, CS0 = CS_MASTER GPIO2_D5; CS1 (GPIO2_D4) = EEPROM MAC locale. 33R serie su CLK/MOSI/MISO verso i connettori."
- note added: "Open drain verso i GPIO PMU: PMIC_INT_L, PD_INT_N (FUSB302B), USB1_OC_N (TPS2553), PWR_SRC_ST (TPS2121) con 10k a VCC3V3_PMU. SD_DET 10k sul foglio Memorie."
- note added: "PHY non usati (USB2 HOST2/3, MULTI_PHY, PCIe3, MIPI CSI/DSI, HDMI, eDP): alimentazioni a VSS e segnali flottanti, secondo 'RK3568 Processing instructions for unused pins'. VDD_NPU su BUCK4 dell'RK809-5."
- note added: "Recovery (ex FEL): SARADC_VIN0 (B27) con 10k a VCCA_1V8 (obbligatorio, Rockchip) e tasto a GND: tenuto premuto all'accensione il loader entra in modalita' Recovery/rockusb."
- note added: "USB3_AVDD_0V9/1V8 da VDDA_0V9/VCCA_1V8 con ferrite 120R@100MHz (reference AIoT), USB3_AVDD_3V3 da VCC_3V3. USB2_AVDD (HOST2/3 non usati) a VSS."
- note added: "USB3_OTG0_DP/DM (porta di flash rkdeveloptool, USB-C di alimentazione) con 2.2R in serie. USB3_HOST1_DP/DM verso la USB-C host (2.2R sul foglio USB host)."
- note added: "VDD_CPU >= 135 uF in totale con le uscite del TCS4525 (Hardware Design Guide 2.2.2.4), un 22 uF DNP di riserva. VDD_LOGIC/GPU/NPU >= 90 uF con le uscite dell'RK809-5."
- note added: "nPOR (AH27, dominio PMUIO1): rete RESETn con 100 nF vicino alla sfera, RESETB dell'RK809-5 (open drain, 10k a VCC3V3_PMU sul foglio PMIC), TSADC_SHUT_M0 con 0R e tasto RESET."
- note removed: "AC_VRA1 su C17 (figura 7-1, footprint EasyEDA e schema Orange Pi Zero2 v1.3; la tabella 4-2 dice D17 per errore). Mappa completa dei pin in docs/pinmap-h616.md."
- note removed: "Analogica (codec e AC300 non usati): VRA1/VRA2 470 nF verso AGND, AGND a GND con 0R, AC_VRA1 1 uF. ZQ del controller DRAM 240R 1% a GND."
- note removed: "CPU: Allwinner H616 (TFBGA-284, 0.65 mm). Ball map solo dal datasheet H616 V1.0 (tabella 4-2, verificata sulla figura 7-1). Serie 3xx."
- note removed: "Clock: quarzo 24 MHz su DXIN/DXOUT (12 pF come la Zero3, da verificare col carico del quarzo scelto; 0R in serie su DXOUT), DXLDO_OUT 220 nF. L'H616 non ha pin per il quarzo 32 kHz: X32KFOUT (PG10) e' derivato internamente."
- note removed: "Come Orange Pi Zero2 (H616) v1.3: REXT (K18) 150k 1% ad AGND (R337), AVCC 2.2 uF (C334), AC_AVCC 10 uF (C335, come la Zero3), AC_VRA1 1 uF su C17."
- note removed: "Disaccoppiamento vicino alle sfere. 100 nF su VCC-PLL, VCC_DCXO, VDD18_DRAM, VCC_HDMI, VCC_TV (VCC-1V8) e su VCC_IO, VCC_PG/PI, VCC_USB, VCC_EPHY (VCC-IO), come la Zero2."
- note removed: "Footprint DNP 10k: pull-up a VCC-1V8-EMMC (= VCC_PC) e pull-down a GND su ogni linea. La Zero3 (boot SPI) usa PC3/PC4/PC6 alti e PC5 basso. Su PC5/PC6 (eMMC) metterli sui via, senza stub."
- note removed: "J301: 1 = TX del SoC (PH0), 2 = RX del SoC (PH1), 3 = GND. Livelli 3.3 V."
- note removed: "Le MISO dei due rami si uniscono dopo i 33R: tutti gli slave (INA239, DAC61402, bus MAIN) devono tenere SDO in alta impedenza con CS alto. ADDR/PREFIX: 100R serie."
- note removed: "Livelli di riposo: CS e CS_MASTER alti (10k), VREF_ENABLE basso (10k a GND), VBIAS_ENABLE basso (100k a GND), ALERT# e HIT# 4.7k, I2C del bus 2.2k, FAULT 10k."
- note removed: "Net DRAM_*/EMMC_*/SD_*/WL_*/BT_*/RGMII_*/PHY_*/GNSS_*/WIFI_*/USB1_*/SPI1_* globali verso gli altri fogli."
- note removed: "P10 WL_REG_ON, P11 BT_REG_ON, P12 BT_WAKE, P13 BT_HOST_WAKE (in), P14 WL_HOST_WAKE (in), P15 SD_DET (in), P16 PHY_EE_CS_N, P17 libera."
- note removed: "Porte: P00 VREF_ENABLE, P01 VBIAS_ENABLE, P02 DAC61402_FAULT (in), P03 USB1_VBUS_EN, P04 VBUS_SRC_EN, P05 PWR_SRC_ST (in), P06 PHY_RST_N, P07 PHY_INT_N (in),"
- note removed: "R336: 3V3_SYS (VDD del FUSB302B) da VCC-IO."
- note removed: "RESET (dominio VCC_PLL 1.8 V): 10k a VCC-1V8 + 1 nF + tasto, 100R in serie dal PWROK dell'AXP313A (AP-RESET), come la Zero3; FEL a GND con tasto (10k a VCC-IO). JTAG_SEL NC come sulla Zero2 (JTAG su PF). PLLTEST, LRADC liberi."
- note removed: "SPI1 (PH6 CLK, PH7 MOSI, PH8 MISO) condiviso tra BUS_POWER e MAIN, chip select con cs-gpios. 33R serie per ramo su CLK/MOSI/MISO; EEPROM MAC locale su SPI1_* (foglio Rete)."
- note removed: "S_TWI0 (PL0/PL1, 1.8 V): AXP313A 0x36, FUSB302B 0x22, TCA6416A 0x20. Pull-up 2.2k a VCC-1V8. Gli open-drain su PC hanno pull-up a VCC-1V8-EMMC (= VCC_PC)."
- note removed: "Strap BOOT_SEL[4:1] = PC6/PC5/PC4/PC3: nessuno montato, come la Zero2 (la tabella livelli -> supporto e' nello User Manual H616 par. 3.4, non disponibile)."
- note removed: "TCA6416A: VCCI = VCC-1V8 (lato I2C), VCCP = VCC-IO (porte a 3.3 V). Al reset tutte le porte sono ingressi: i pull-up/pull-down esterni fissano lo stato sicuro."
