File: SchedaH616/progetto-kicad/gnss.kicad_sch (KiCad schematic)
At the start: 26 parts, among them J701 SMA antenna, J702 SMA PPS OUT, J703 SMA STROBE IN, J704 PPS/STROBE, U701 NEO-M9N-00B, U702 74LVC1G17, U703 74LVC1G17

Commit message: SchedaH616: placement PCB 50x70 a 6 strati e modifiche allo schema
PCB (solo placement, niente piste), generato da generatori/build_pcb.sh:
- 50 x 70 mm, smussi 3 mm, 4 fori NPTH 2.2 mm con keepout, 6 strati
- H616 al centro, LPDDR4 sul lato DRAM, AXP313A vicino alla CPU, eMMC vicino ai pin PC
- connettori sui bordi, U.FL Wi-Fi e SMA GNSS su lati opposti
- disaccoppiamento di H616 e LPDDR4 sul bottom sotto le sfere
- regole: piste 5 mil, via-in-pad 0.25/0.15 sotto l'H616
- DRC: 0 violazioni (solo collegamenti da fare), parità schema/PCB ok

Schema (modifiche approvate):
- LPDDR4 confermata come scelta definitiva
- USB host di nuovo su USB-C solo host (Rp 22k, USBLC6-2, TPS2553)
- jack 5 V diretto su IN1 del TPS2121, tolto l'SS54, TPS56637 in Eco-mode
- LDO AP2112K-1.8 (C176944) dedicato a VCCQ eMMC e VCC_PC
- ERC 0

Libreria H616.pretty: serigrafia sui pad tolta, pioli di centraggio NPTH.

Co-Authored-By: Claude Opus 5.5 (1M context) <noreply@anthropic.com>
Parts:
- TP701, TP702: now left out of the parts list

Commit message: SchedaH616: RK3568 + RK809-5 + TCS4525 + DDR4, placement 50x70
- SoC Allwinner H616 -> Rockchip RK3568 (FCBGA636L, LCSC C2938930): ball map dal pinout
  Rockchip V1.1, verificata sulla tabella 2-1 del datasheet V1.2 (636/636); footprint
  generato (gen_fp.py), confrontato con EasyEDA C2938930
- PMIC AXP313A -> RK809-5 (C2939628) come Rockchip AIoT REF V1.1 / ROCK 3A; TCS4525 per
  VDD_CPU su I2C0 (0x1C); BUCK4 su VDD_NPU (sull'RK809-5 parte spento: non puo' fare il 3.3 V)
- LPDDR4 -> DDR4 x16 K4AAG165WA-BCWE (C2920140) sul canale A, point-to-point, niente VTT,
  VPP da AP2112K-2.5, ZQ 240R, DDR_RZQ del SoC 120R (Hardware Design Guide)
- eMMC su EMMC 8 bit (VCCIO2 1.8 V), microSD su SDMMC0, AP6256 su SDMMC2 + UART8,
  RTL8211F su GMAC0 RGMII (22R TX al SoC e RX al PHY), console UART2_M0, USB-C su OTG0
- Recovery su SARADC_VIN0, reset sulla rete RESETn; TCA6416A tolto
- Bus MIKILAB: BUS_POWER su SPI3_M1, MAIN su SPI2_M1 (CS del DAC su cs-gpios)
- progetto rinominato SchedaRK3568, libreria di progetto Scheda; script portabili Linux/macOS
- ERC 0, parita' 0, DRC 0 (solo collegamenti da fare); placement 439/439

Co-Authored-By: Claude Opus 5.5 (1M context) <noreply@anthropic.com>
Parts:
- BT701: footprint H616:BatteryHolder_MYOUNG_BS-12-B3AA003_CR1220 -> Scheda:BatteryHolder_MYOUNG_BS-12-B3AA003_CR1220
Connections:
- net 3V3_PERI renamed VCC_3V3
- net GNSS_UART2_RX renamed GNSS_UART_RX
- net GNSS_UART2_TX renamed GNSS_UART_TX
Other:
- note added: "Alimentazione: VCC 10uF + 0.1uF. Backup V_BCKP da OR di diodi: VCC_3V3 (BAT54) e pila CR1220 (BAT54), nessuna ricarica della pila."
- note added: "UART3_M1: TXD del modulo -> GNSS_UART_RX (GPIO3_C0), RXD <- GNSS_UART_TX (GPIO3_B7). TIMEPULSE -> 33R -> GNSS_PPS (GPIO3_A5). EXTINT (pin 4, PIO7, time mark TIM-TM2) letto anche da GPIO3_A6 (solo ingresso)."
- note removed: "Alimentazione: VCC 10uF + 0.1uF. Backup V_BCKP da OR di diodi: 3V3_PERI (BAT54) e pila CR1220 (BAT54), nessuna ricarica della pila."
- note removed: "UART2: TXD del modulo -> GNSS_UART2_RX (PG16), RXD <- GNSS_UART2_TX (PG15). TIMEPULSE -> 33R -> GNSS_PPS (PG13, EINT). EXTINT (pin 4, PIO7, time mark TIM-TM2) letto anche da PG14 (EINT, solo ingresso)."
