File: SchedaH616/progetto-kicad/gnss.kicad_sch (KiCad schematic)
At the start: 26 parts, among them J701 SMA antenna, J702 SMA PPS OUT, J703 SMA STROBE IN, J704 PPS/STROBE, U701 NEO-M9N-00B, U702 74LVC1G17, U703 74LVC1G17

Commit message: SchedaH616: passivi 0603, microSD sul bottom, USB-C affiancate
- passivi 0603 di default; 0201/0402 solo per il disaccoppiamento sotto RK3568 e DDR4,
  le serie RGMII/clock/USB, DDR_RZQ, ZQ e VREF della DDR4
  (C: 29x0201, 31x0402, 133x0603; R: 24x0402, 133x0603)
- microSD J401 sul bottom, apertura sul bordo sinistro
- USB-C host J801 e OTG/alimentazione J104 affiancate sul bordo basso, con ESD,
  TPS2553, TPS2121, FUSB302B e SY6280 accanto
- 387 componenti sul top, 52 sul bottom; ERC 0, parita' 0, DRC 0 (solo collegamenti)

Co-Authored-By: Claude Opus 5.5 (1M context) <noreply@anthropic.com>
Parts:
- C702, C703, C704, C705, C706: footprint Capacitor_SMD:C_0402_1005Metric -> Capacitor_SMD:C_0603_1608Metric
- R702, R703, R704, R705, R706: footprint Resistor_SMD:R_0402_1005Metric -> Resistor_SMD:R_0603_1608Metric
