File: SchedaH616/progetto-kicad/pmic.kicad_sch (KiCad schematic)
At the start: 33 parts, among them U201 AXP313A, U202 TPS563201DDCR

Commit message: SchedaH616: placement PCB 50x70 a 6 strati e modifiche allo schema
PCB (solo placement, niente piste), generato da generatori/build_pcb.sh:
- 50 x 70 mm, smussi 3 mm, 4 fori NPTH 2.2 mm con keepout, 6 strati
- H616 al centro, LPDDR4 sul lato DRAM, AXP313A vicino alla CPU, eMMC vicino ai pin PC
- connettori sui bordi, U.FL Wi-Fi e SMA GNSS su lati opposti
- disaccoppiamento di H616 e LPDDR4 sul bottom sotto le sfere
- regole: piste 5 mil, via-in-pad 0.25/0.15 sotto l'H616
- DRC: 0 violazioni (solo collegamenti da fare), parità schema/PCB ok

Schema (modifiche approvate):
- LPDDR4 confermata come scelta definitiva
- USB host di nuovo su USB-C solo host (Rp 22k, USBLC6-2, TPS2553)
- jack 5 V diretto su IN1 del TPS2121, tolto l'SS54, TPS56637 in Eco-mode
- LDO AP2112K-1.8 (C176944) dedicato a VCCQ eMMC e VCC_PC
- ERC 0

Libreria H616.pretty: serigrafia sui pad tolta, pioli di centraggio NPTH.

Co-Authored-By: Claude Opus 5.5 (1M context) <noreply@anthropic.com>
Parts:
- added C222, C223: 1uF/10V, Capacitor_SMD:C_0402_1005Metric, symbol Device:C
- added U203: AP2112K-1.8TRG1, Package_TO_SOT_SMD:SOT-23-5, symbol Regulator_Linear:AP2112K-1.8
- TP201: now left out of the parts list
Connections:
- net 3V3_PERI: now also C222.1, U203.1 (VIN), U203.3 (EN)
- net GND_D: now also C222.2, C223.2, U203.2 (GND)
- new net VCC-1V8-EMMC: C223.1, U203.5 (VOUT)
- no-connect marks 3 -> 4
Other:
- note added: "ALDO1 VCC-1V8 300 mA (VCC_PLL, VDD18_DRAM, DCXO, AVCC, AC_AVCC, HDMI, TV, LPDDR4 VDD1, TCA6416A VCCI), DLDO1 VCC-IO 3.3 V 500 mA (VCC_IO/PG/PI/USB). RTCLDO non usato (H616 senza VCC_RTC)."
- note added: "EN legato a VIN: parte con 3V3_PERI, cioe' dopo DLDO1 (EN del TPS563201 da VCC-IO). 1 uF in ingresso e in uscita."
- note added: "VCC-1V8-EMMC: LDO AP2112K-1.8TRG1 (LCSC C176944, 600 mA) da 3V3_PERI per VCCQ eMMC (fino a ~132 mA in HS400) e VCC_PC dell'H616: banco PC ed eMMC salgono insieme. Scarica ALDO1."
- note removed: "ALDO1 VCC-1V8 300 mA (VCC_PLL, VDD18_DRAM, DCXO, AVCC, VCC_PC/eMMC VCCQ, LPDDR4 VDD1), DLDO1 VCC-IO 3.3 V 500 mA (VCC_IO/PG/PI/USB). RTCLDO non usato (H616 senza VCC_RTC)."

Commit message: SchedaH616: verifica sullo schema Orange Pi Zero3 (LPDDR4, AXP313A, reset)
- Mappa CA/CS/CK/CKE/RESET della LPDDR4 verificata 8/8 sulla Zero3, sfere della LPDDR4, ODT 100k e ZQ 240R coincidono
- AXP313A allineato alla Zero3: 22 uF sui VIN, 2x47 uF + 1 uF + 100 nF sulle uscite DCDC, DLDO1 47 uF, RTCLDO 4.7 uF, PWRON 100 nF montato
- DCDC3 a 1.1 V impostato dall'SPL di U-Boot (CONFIG_AXP_DCDC3_VOLT)
- RESET H616: 10k a VCC-1V8, 1 nF, 100R in serie da AP-RESET; AC_AVCC 10 uF; quarzo 24 MHz con 12 pF
- scelte-progetto.md: verifiche segnate, differenze volute (VCC_PG 3.3 V, VCC_PC 1.8 V), nuovo punto aperto sugli strap BOOT_SEL
- ERC 0, parita' 0, DRC 0 (solo collegamenti da fare)

Co-Authored-By: Claude Opus 5.5 (1M context) <noreply@anthropic.com>
Parts:
- added C224, C225: 1uF, Capacitor_SMD:C_0402_1005Metric, symbol Device:C
- added C226, C227, C228, C230: 100nF, Capacitor_SMD:C_0402_1005Metric, symbol Device:C
- added C229: 47uF/6.3V, Capacitor_SMD:C_0603_1608Metric, symbol Device:C
- added C231: 4.7uF/10V, Capacitor_SMD:C_0402_1005Metric, symbol Device:C
- C201, C202, C203: value 10uF/10V -> 22uF/10V
- C208, C209, C210, C211, C212: value 22uF/6.3V -> 47uF/6.3V
- C213: value 22uF/6.3V -> 1uF; footprint Capacitor_SMD:C_0603_1608Metric -> Capacitor_SMD:C_0402_1005Metric
- C215: value 4.7uF/10V -> 47uF/6.3V; footprint Capacitor_SMD:C_0402_1005Metric -> Capacitor_SMD:C_0603_1608Metric
- C216: now fitted
Connections:
- net GND_D: now also C224.2, C225.2, C226.2, C227.2, C228.2, C229.2, C230.2, C231.2
- net VCC-DRAM: now also C229.1, C230.1
- net VCC-IO: now also C226.1
- net VDD-CPU: now also C225.1, C228.1
- net VDD-SYS: now also C224.1, C227.1
- net PMU_RTCLDO: now reaches U201.7 (RTCLDO)
- net PMU_RTCLDO: now also C231.1
- no-connect marks 4 -> 3
Other:
- note added: "Controllo: PWROK = AP-RESET -> 100R -> RESET del SoC (foglio CPU), pull-up 10k a VCC-1V8. Accensione all'arrivo di VIN; PWRON su test point. IRQ non collegato (la Zero3 lo porta su PC9 con 0R; qui non ci sono GPIO liberi sicuri: PC3/PC4 sono strap BOOT_SEL)."
- note added: "Ingressi VIN1/VIN2/VIN3: 22 uF + 100 nF ciascuno vicino ai pin (Zero3: 22 uF). Pin 8 (VREF, GPO sulla Zero3) 1 uF."
- note added: "Uscite come la Zero3: VDD-GPU/SYS e VDD-CPU 2x47 uF + 1 uF + 100 nF, VCC-DRAM 2x47 uF + 1 uF + 100 nF, DLDO1 47 uF + 100 nF, RTCLDO 4.7 uF (non usato dall'H616). DCDC: induttori 1 uH (datasheet: Isat > 1.3 x carico, DCR < 30 mohm), uscite >= 10 uF. FB con sense remoto: DCDC1 da VDD_GPUFB (F8), DCDC2 da VDD_CPUFB (L8), DCDC3 dalla LPDDR4."
- note removed: "Controllo: PWROK -> RESET del SoC (dominio VCC_PLL 1.8 V), pull-up 10k a VCC-1V8. Accensione all'arrivo di VIN; PWRON su test point. IRQ non collegato (nessun GPIO libero)."
- note removed: "DCDC: induttori 1 uH (datasheet: Isat > 1.3 x carico, DCR < 30 mohm), uscite >= 10 uF. FB con sense remoto: DCDC1 da VDD_GPUFB (F8), DCDC2 da VDD_CPUFB (L8), DCDC3 dalla LPDDR4."
- note removed: "Ingressi VIN1/VIN2/VIN3: 10 uF + 100 nF ciascuno vicino ai pin. VREF 1 uF (datasheet)."

Commit message: SchedaH616: RK3568 + RK809-5 + TCS4525 + DDR4, placement 50x70
- SoC Allwinner H616 -> Rockchip RK3568 (FCBGA636L, LCSC C2938930): ball map dal pinout
  Rockchip V1.1, verificata sulla tabella 2-1 del datasheet V1.2 (636/636); footprint
  generato (gen_fp.py), confrontato con EasyEDA C2938930
- PMIC AXP313A -> RK809-5 (C2939628) come Rockchip AIoT REF V1.1 / ROCK 3A; TCS4525 per
  VDD_CPU su I2C0 (0x1C); BUCK4 su VDD_NPU (sull'RK809-5 parte spento: non puo' fare il 3.3 V)
- LPDDR4 -> DDR4 x16 K4AAG165WA-BCWE (C2920140) sul canale A, point-to-point, niente VTT,
  VPP da AP2112K-2.5, ZQ 240R, DDR_RZQ del SoC 120R (Hardware Design Guide)
- eMMC su EMMC 8 bit (VCCIO2 1.8 V), microSD su SDMMC0, AP6256 su SDMMC2 + UART8,
  RTL8211F su GMAC0 RGMII (22R TX al SoC e RX al PHY), console UART2_M0, USB-C su OTG0
- Recovery su SARADC_VIN0, reset sulla rete RESETn; TCA6416A tolto
- Bus MIKILAB: BUS_POWER su SPI3_M1, MAIN su SPI2_M1 (CS del DAC su cs-gpios)
- progetto rinominato SchedaRK3568, libreria di progetto Scheda; script portabili Linux/macOS
- ERC 0, parita' 0, DRC 0 (solo collegamenti da fare); placement 439/439

Co-Authored-By: Claude Opus 5.5 (1M context) <noreply@anthropic.com>
Parts:
- removed U201: AXP313A, H616:QFN-20_L3.0-W3.0-P0.40-BL-EP1.7, symbol H616:AXP313A
- removed U202: TPS563201DDCR, Package_TO_SOT_SMD:SOT-23-6, symbol Regulator_Switching:TPS563201
- removed U203: AP2112K-1.8TRG1, Package_TO_SOT_SMD:SOT-23-5, symbol Regulator_Linear:AP2112K-1.8
- added C232, C233, C234, C236, C237, C238, C239, C248: 1uF, Capacitor_SMD:C_0402_1005Metric, symbol Device:C
- added C235: 10uF/10V, Capacitor_SMD:C_0603_1608Metric, symbol Device:C
- added C240, C241: 22pF, Capacitor_SMD:C_0402_1005Metric, symbol Device:C
- added C242, C243, C244, C247, C254, C255, C263, C264: 100nF, Capacitor_SMD:C_0402_1005Metric, symbol Device:C
- added C245, C246, C256, C257: 22uF/10V, Capacitor_SMD:C_0805_2012Metric, symbol Device:C
- added C249, C250, C251, C252: 22uF, Capacitor_SMD:C_0603_1608Metric, symbol Device:C
- added C253: 10uF/16V, Capacitor_SMD:C_0805_2012Metric, symbol Device:C
- added C258, C259, C260: 1uF/10V, Capacitor_SMD:C_0402_1005Metric, symbol Device:C
- added C261, C262: 4.7uF, Capacitor_SMD:C_0402_1005Metric, symbol Device:C
- added L205: 0.47uH/4A, Inductor_SMD:L_1008_2520Metric, symbol Device:L
- added L206: 0.33uH/9A, Inductor_SMD:L_Coilcraft_XAL4020-XXX, symbol Device:L
- added L207: 2.2uH/4A, Inductor_SMD:L_Coilcraft_XAL4020-XXX, symbol Device:L
- added R206, R207: 22R, Resistor_SMD:R_0402_1005Metric, symbol Device:R
- added R208, R210: 10k, Resistor_SMD:R_0402_1005Metric, symbol Device:R
- added R209: 0R, Resistor_SMD:R_0402_1005Metric, symbol Device:R
- added R211, R215: 100k, Resistor_SMD:R_0402_1005Metric, symbol Device:R
- added R212: 22k, Resistor_SMD:R_0402_1005Metric, symbol Device:R
- added R213: 51k, Resistor_SMD:R_0402_1005Metric, symbol Device:R
- added R214: 100R, Resistor_SMD:R_0402_1005Metric, symbol Device:R
- added R216: 33.2k 1%, Resistor_SMD:R_0402_1005Metric, symbol Device:R
- added R217: 10k 1%, Resistor_SMD:R_0402_1005Metric, symbol Device:R
- added TP202: PWRON, TestPoint:TestPoint_Pad_D1.0mm, symbol Connector:TestPoint
- added U201: RK809-5, Package_DFN_QFN:ArtInChip_QFN-68-1EP_7x7mm_P0.35mm_EP5.49x5.49mm, symbol Scheda:RK809-5
- added U202: TCS4525_WT, Package_CSP:DiodesInc_GEA20_WLCSP-20_1.7x2.1mm_Layout4x5_P0.4mm, symbol Scheda:TCS4525
- added U203: TPS563201DDCR, Package_TO_SOT_SMD:SOT-23-6, symbol Regulator_Switching:TPS563201
- added U204: AP2112K-1.8TRG1, Package_TO_SOT_SMD:SOT-23-5, symbol Regulator_Linear:AP2112K-1.8
- added U205: AP2112K-2.5TRG1, Package_TO_SOT_SMD:SOT-23-5, symbol Regulator_Linear:AP2112K-2.5
- added Y201: 32.768kHz, Crystal:Crystal_SMD_3215-2Pin_3.2x1.5mm, symbol Device:Crystal
- C202, C203: value 22uF/10V -> 10uF/10V
- C204: value 100nF -> 10uF/10V; footprint Capacitor_SMD:C_0402_1005Metric -> Capacitor_SMD:C_0603_1608Metric
- C205, C206, C226, C227, C230: value 100nF -> 1uF
- C207: value 1uF/10V -> 1uF
- C208, C210, C229: value 47uF/6.3V -> 1uF; footprint Capacitor_SMD:C_0603_1608Metric -> Capacitor_SMD:C_0402_1005Metric
- C209, C211: value 47uF/6.3V -> 10uF/10V
- C212, C215: value 47uF/6.3V -> 22uF
- C213, C224: value 1uF -> 22uF; footprint Capacitor_SMD:C_0402_1005Metric -> Capacitor_SMD:C_0603_1608Metric
- C214: value 4.7uF/10V -> 100nF
- C216, C218: value 100nF -> 22uF; footprint Capacitor_SMD:C_0402_1005Metric -> Capacitor_SMD:C_0603_1608Metric
- C217: value 10uF/16V -> 100nF; footprint Capacitor_SMD:C_0805_2012Metric -> Capacitor_SMD:C_0402_1005Metric
- C219: value 100nF -> 10uF; footprint Capacitor_SMD:C_0402_1005Metric -> Capacitor_SMD:C_0603_1608Metric
- C220, C221: value 22uF/10V -> 22uF; footprint Capacitor_SMD:C_0805_2012Metric -> Capacitor_SMD:C_0603_1608Metric
- C222: value 1uF/10V -> 100nF
- C223: value 1uF/10V -> 22uF; footprint Capacitor_SMD:C_0402_1005Metric -> Capacitor_SMD:C_0603_1608Metric
- C228: value 100nF -> 4.7uF
- C231: value 4.7uF/10V -> 1uF
- L201: value 1uH/2.5A -> 0.47uH/4A; MPN 1uH 2.5A DCR<30m -> TFM252012ALMA-R47MTAA
- L202: value 1uH/4A -> 0.47uH/4A; footprint Inductor_SMD:L_Coilcraft_XAL4020-XXX -> Inductor_SMD:L_1008_2520Metric; MPN XAL4020-102 -> TFM252012ALMA-R47MTAA
- L203: value 1uH/3A -> 0.47uH/4A; MPN 1uH 3A DCR<30m -> TFM252012ALMA-R47MTAA
- L204: value 2.2uH/4A -> 0.47uH/4A; footprint Inductor_SMD:L_Coilcraft_XAL4020-XXX -> Inductor_SMD:L_1008_2520Metric; MPN XAL4020-222 -> TFM252012ALMA-R47MTAA
- R201: value 10k -> 0R
- R202: value 0R -> 62k 1%
- R203: value 100k -> 120k 1%; now fitted
- R204: value 33.2k 1% -> 0R
- R205: value 10k 1% -> DNP; now not fitted
- TP201: value PWRON -> VCC_1V8
Connections:
- net VCC-1V8-EMMC is gone; now on net VCC_1V8: C223.1
- net 5V_SYS: now also C245.1, C246.1, C253.1, C254.1, R211.1, R215.1, U202.D1 (AVIN), U202.D2 (PVIN), U202.E1 (PVIN), U202.E2 (PVIN), U203.3 (VIN); no longer C201.1, C202.1, C203.1, C204.1, C205.1, C206.1, C217.1, C218.1, R203.1
- net GND_D: now also C219.2, R203.2, C232.2, C233.2, C234.2, C235.2, C236.2, C237.2, C238.2, C239.2, C240.2, C241.2, C242.2, C243.2, C244.2, C245.2, C246.2, C247.2, C248.2, C249.2, C250.2, C251.2, C252.2, C253.2, C254.2, C256.2, C257.2, C258.2, C259.2, C260.2, C261.2, C262.2, C263.2, C264.2, R212.2, R217.2, U201.14 (LRCLK), U201.15 (BCLK), U201.16 (MCLK), U201.17 (SDI), U201.19 (PDMCLK), U201.40 (HP_SNS), U201.47 (GNDREF), U201.56 (BATDIV), U201.62 (SNSP), U201.63 (SNSN), U201.69 (EPAD), U202.B2 (PGND), U202.B3 (PGND/PG), U202.B4 (AGND), U202.C1 (PGND), U202.C2 (PGND), U202.C3 (PGND), U202.C4 (PGND), U203.1 (GND), U204.2 (GND), U205.2 (GND)
- net PERI_BST: now also C255.1, U203.6 (VBST); no longer C219.1
- net PERI_EN: now also R215.2, U203.5 (EN); no longer R202.2, R203.2
- net PERI_FB: now also R216.2, R217.1, U203.4 (VFB); no longer R204.2, R205.1
- net PERI_SW: now also C255.2, L207.1, U203.2 (SW); no longer C219.2, L204.1
- net 3V3_PERI renamed VDD_NPU
- net VDD_NPU: now also U201.64 (FB4); no longer R204.1
- net AP-RESET renamed PMIC_VCC_SPK
- net PMIC_VCC_SPK: now also C211.1, U201.33 (VCC_SPK_HP)
- net PMU_LX1 renamed PMIC_SW1
- net PMIC_SW1: now also U201.12 (SW1)
- net PMU_LX2 renamed PMIC_SW2
- net PMIC_SW2: now also U201.9 (SW2)
- net PMU_LX3 renamed PMIC_SW3
- net PMIC_SW3: now also U201.25 (SW3)
- net PMU_PWRON renamed VCC_1V8
- net VCC_1V8: now also C224.1, R204.1, L205.2; no longer C216.1
- net PMU_RTCLDO renamed VCCA_1V8
- net VCCA_1V8: now also U201.3 (LDO7)
- net PMU_VREF renamed VCC3V3_SYS
- net VCC3V3_SYS: now also C201.1, C202.1, C203.1, C204.1, C205.1, C206.1, C208.1, C209.1, C210.1, R201.1, C239.1, C256.1, C257.1, C258.1, C260.1, L207.2, R216.1, U201.10 (VCC2), U201.11 (VCC1), U201.22 (VCC5), U201.24 (VCC3), U201.30 (VCC6), U201.4 (VCC7), U201.45 (VCC_RTC), U201.54 (VCC9), U201.57 (VCC8), U201.66 (VCC4), U204.1 (VIN), U205.1 (VIN)
- net VCC-1V8 renamed VDD_LOGIC
- net VDD_LOGIC: now also C212.1, C213.1, L201.2, U201.13 (FB1); no longer R201.1
- removed net VCC-DRAM: C212.1, C213.1, C229.1, C230.1, L203.2
- removed net VCC-IO: C215.1, C226.1, R202.1
- removed net VDD-CPU: C210.1, C211.1, C225.1, C228.1, L202.2
- removed net VDD-SYS: C208.1, C209.1, C224.1, C227.1, L201.2
- new net CLK32K: R209.2, R210.2
- new net I2C0_SCL: R207.1, U202.A3 (SCL)
- new net I2C0_SDA: R206.1, U202.B1 (SDA)
- new net PMIC_1P8A: C237.1, U201.44 (VCC_1P8A)
- new net PMIC_1P8D: C238.1, U201.48 (VCC_1P8D)
- new net PMIC_CLK32K: R209.1, U201.68 (CLK32K)
- new net PMIC_FB3: R202.2, R203.1, U201.27 (FB3)
- new net PMIC_FB5: R204.2, R205.1, U201.59 (FB5)
- new net PMIC_INT_L: U201.7 (INT)
- new net PMIC_LDO1: C225.1, U201.23 (LDO1)
- new net PMIC_LDO4: C228.1, U201.28 (LDO4)
- new net PMIC_LDO9: C233.1, U201.6 (LDO9)
- new net PMIC_PWRON: C243.1, TP202.1, U201.52 (PWRON)
- new net PMIC_SCL: R207.2, U201.1 (SCL)
- new net PMIC_SDA: R206.2, U201.2 (SDA)
- new net PMIC_SLEEP_H: U201.49 (SLEEP), U202.A1 (VSEL)
- new net PMIC_SW4: L204.1, U201.65 (SW4)
- new net PMIC_SW5: L205.1, U201.53 (SW5)
- new net PMIC_VDC: C244.1, R211.2, R212.1, U201.61 (VDC)
- new net PMIC_VREF: C236.1, U201.46 (VREF)
- new net PMIC_XIN: C240.1, U201.50 (XIN), Y201.1
- new net PMIC_XOUT: C241.1, U201.51 (XOUT), Y201.2
- new net RESETn: C242.1, R208.2, U201.67 (RESETB)
- new net TCS_EN: C247.1, R213.2, U202.A2 (EN)
- new net TCS_SW: L206.1, U202.D3 (SW), U202.D4 (SW), U202.E3 (SW), U202.E4 (SW)
- new net VCC1V8_EMMC: C259.1, U204.5 (VOUT)
- new net VCC2V5_DDR: C261.1, C262.1, C263.1, C264.1, U205.5 (VOUT)
- new net VCC3V3_PMU: C230.1, R208.1, R210.1, R213.1, U201.31 (LDO6), U204.3 (EN), U205.3 (EN)
- new net VCC3V3_SD: C234.1, U201.58 (SWOUT2)
- new net VCCA1V8_PMU: C232.1, U201.5 (LDO8)
- new net VCCIO_SD: C229.1, U201.29 (LDO5)
- new net VCC_3V3: C235.1, U201.55 (SWOUT1)
- new net VCC_DDR: C218.1, C219.1, L203.2, R202.1, U201.26 (VBUCK3)
- new net VDDA0V9_PMU: C227.1, U201.20 (LDO3)
- new net VDDA_0V9: C226.1, U201.21 (LDO2)
- new net VDD_CPU: C248.1, C249.1, C250.1, C251.1, C252.1, L206.2, R214.1
- new net VDD_CPU_COM: R214.2, U202.A4 (FB)
- new net VDD_GPU: C215.1, C216.1, C217.1, L202.2, U201.8 (FB2)
- no-connect marks 3 -> 14
Other:
- note added: "BUCK3 VCC_DDR = 0.8 V x (1 + 62k/120k) = 1.21 V per DDR4 (tabella del reference: DDR4 1.21 V con 62K 1%)."
- note added: "BUCK4 parte spento a 0.5 V: non puo' essere il 3.3 V di sistema (resterebbe tutto spento). Il 3.3 V resta sul TPS563201 (VCC3V3_SYS) come nel reference Rockchip; BUCK4 alimenta VDD_NPU (come ROCK 3A)."
- note added: "BUCK5 VCC_1V8 (1.8 V, seq 2) libero: la VCCQ dell'eMMC e VCCIO2 restano sull'AP2112K-1.8 come richiesto. Test point TP201."
- note added: "BUCK: induttori 0.47 uH 2520 (DCR < 50 mohm, datasheet: 0.47 uH/4 A BUCK1/2/5, 3 A BUCK3/4). FB1/FB2/FB4 sulle uscite (VDD_LOGIC/GPU/NPU), come il reference."
- note added: "Codec non usato (nota del reference): pin 14, 15, 16, 17, 19, 40 a VSS; 18, 32, 34-39, 41-43 flottanti. VCC_SPK_HP (33) da VCC3V3_SYS: il datasheet chiede VCC_RTC (45) = tensione piu' alta dell'RK809."
- note added: "Default RK809-5 (tabella 4-4): BUCK1 0.9 V seq 1, BUCK2 0.9 V seq 2, BUCK3 da partitore seq 3, BUCK4 SPENTO (0.5 V), BUCK5 1.8 V seq 2, LDO2/3 0.9 V seq 1, LDO5 3.3 V seq 4, LDO6 3.3 V seq 2, LDO7/8 1.8 V seq 2, SWOUT1/2 seq 4."
- note added: "FB (A4) = VDD_CPU_COM (sfera M15 del SoC, sense remoto) con 100R verso VDD_CPU. Induttore 0.33 uH (datasheet: 0.33 o 0.47 uH), Isat > 8 A (picco 8 A). PGND/PG (B3) a GND."
- note added: "Gestione: VREF 1 uF, VCC_1P8A/1P8D 1 uF, VCC_RTC 1 uF, quarzo 32.768 kHz Y201 con 2x 22 pF (reference). SDA/SCL 22R serie verso I2C0."
- note added: "Ingressi (reference AIoT): VCC1 22 uF, VCC2/VCC3/VCC4/VCC9 10 uF, VCC5-VCC8 1 uF, tutti vicino ai pin."
- note added: "LDO e switch (reference AIoT): 1 uF su ogni uscita, LDO4 4.7 uF, SWOUT1 10 uF. LDO1/LDO4/LDO9 (IMAGE, ACODEC) non usati: spenti di default, solo il condensatore."
- note added: "LDO2 VDDA_0V9, LDO3 VDDA0V9_PMU, LDO5 VCCIO_SD (VCCIO3), LDO6 VCC3V3_PMU (PMUIO1/2), LDO7 VCCA_1V8, LDO8 VCCA1V8_PMU, SWOUT1 VCC_3V3 (VCCIO4-7 e periferiche), SWOUT2 VCC3V3_SD (microSD)."
- note added: "PMIC RK809-5 (datasheet Rockchip RK809 Rev 2.3; schema come Rockchip RK3568 AIoT REF V1.1 pag. 22 e Radxa ROCK 3A): ingressi VCC1-VCC9 da VCC3V3_SYS, I2C0 0x20. Serie 2xx."
- note added: "PWRON con 100 nF e test point (accensione a mano). VDC: partitore da 5V_SYS, la PMIC parte da sola quando arriva l'alimentazione."
- note added: "RESETB -> RESETn (nPOR del SoC) con 10k a VCC3V3_PMU e 100 nF. CLK32K (open drain) -> 0R -> CLK32K: CLK32K_IN del SoC (GPIO0_B0) e LPO dell'AP6256, 10k a VCC3V3_PMU."
- note added: "VCC1V8_EMMC: AP2112K-1.8TRG1 (LCSC C176944) da VCC3V3_SYS per VCCQ dell'eMMC e VCCIO2 (FLASH_VOL_SEL alto). EN da VCC3V3_PMU: sale con la sequenza della PMIC."
- note added: "VCC2V5_DDR (VPP della DDR4): AP2112K-2.5TRG1 da VCC3V3_SYS, EN da VCC3V3_PMU (seq 2, prima di VCC_DDR seq 3: VPP >= VDD come chiede JEDEC). Uscita 2x 4.7 uF + 2x 100 nF (reference)."
- note added: "VCC3V3_SYS: TPS563201 da 5V_SYS, 3.3 V / 3 A, sempre acceso (EN 100k a 5V_SYS). Alimenta RK809-5 (VCC1-9), FUSB302B e i due LDO. Le periferiche stanno su VCC_3V3 (SWOUT1)."
- note added: "VCC_RTC (45) a VCC3V3_SYS con 1 uF (fig. 1-2 del datasheet, senza batteria). VDC (61) da 5V_SYS con 100k/22k = 0.9 V (>0.55 V: accensione al fronte di salita). BATDIV/SNSP/SNSN a GND. EXT_EN libero."
- note added: "VDD_CPU: TCS4525 (datasheet TCS Ver.1.0) come reference AIoT pag. 23 e ROCK 3A: VIN da 5V_SYS, I2C0 0x1C, VSEL da PMIC_SLEEP_H, EN da VCC3V3_PMU con 51k (parte dopo LDO6)."
- note added: "Vout = 0.768 V x (1 + 33.2k/10k) = 3.32 V. Carico stimato 2.5-3 A di picco (bucks RK809 + SWOUT1/2): al limite dei 3 A, vedi punti aperti."
- note removed: "3V3_PERI: TPS563201 da 5V_SYS, 3.3 V / 3 A per AP6256 (VBAT), RTL8211F, NEO-M9N, eMMC VCC, microSD, EEPROM MAC. EN da VCC-IO (parte dopo DLDO1)."
- note removed: "ALDO1 VCC-1V8 300 mA (VCC_PLL, VDD18_DRAM, DCXO, AVCC, AC_AVCC, HDMI, TV, LPDDR4 VDD1, TCA6416A VCCI), DLDO1 VCC-IO 3.3 V 500 mA (VCC_IO/PG/PI/USB). RTCLDO non usato (H616 senza VCC_RTC)."
- note removed: "Controllo: PWROK = AP-RESET -> 100R -> RESET del SoC (foglio CPU), pull-up 10k a VCC-1V8. Accensione all'arrivo di VIN; PWRON su test point. IRQ non collegato (la Zero3 lo porta su PC9 con 0R; qui non ci sono GPIO liberi sicuri: PC3/PC4 sono strap BOOT_SEL)."
- note removed: "DCDC1 VDD-SYS 0.9 V (VDD_SYS + VDD_GPU, max 0.99 V) 1.5 A, DCDC2 VDD-CPU 0.81-1.1 V 3 A, DCDC3 VCC-DRAM 1.1 V (LPDDR4 VDD2/VDDQ) 2 A,"
- note removed: "EN legato a VIN: parte con 3V3_PERI, cioe' dopo DLDO1 (EN del TPS563201 da VCC-IO). 1 uF in ingresso e in uscita."
- note removed: "Ingressi VIN1/VIN2/VIN3: 22 uF + 100 nF ciascuno vicino ai pin (Zero3: 22 uF). Pin 8 (VREF, GPO sulla Zero3) 1 uF."
- note removed: "LDO: ALDO1 VCC-1V8 e DLDO1 VCC-IO con 4.7 uF (datasheet: >= 1 uF). RTCLDO libero (LDO non usato: pin flottante, nessun condensatore)."
- note removed: "PMIC AXP313A (datasheet X-Powers v1.0) come su Orange Pi Zero3 (H618 + AXP313A): VIN 3.0-5.5 V da 5V_SYS, I2C 0x36 su S_TWI0 (PL0/PL1). Serie 2xx."
- note removed: "Uscite come la Zero3: VDD-GPU/SYS e VDD-CPU 2x47 uF + 1 uF + 100 nF, VCC-DRAM 2x47 uF + 1 uF + 100 nF, DLDO1 47 uF + 100 nF, RTCLDO 4.7 uF (non usato dall'H616). DCDC: induttori 1 uH (datasheet: Isat > 1.3 x carico, DCR < 30 mohm), uscite >= 10 uF. FB con sense remoto: DCDC1 da VDD_GPUFB (F8), DCDC2 da VDD_CPUFB (L8), DCDC3 dalla LPDDR4."
- note removed: "VCC-1V8-EMMC: LDO AP2112K-1.8TRG1 (LCSC C176944, 600 mA) da 3V3_PERI per VCCQ eMMC (fino a ~132 mA in HS400) e VCC_PC dell'H616: banco PC ed eMMC salgono insieme. Scarica ALDO1."
- note removed: "Vout = 0.768 V x (1 + R204/R205) = 3.32 V. R203 DNP: alternativa per accenderlo sempre da 5V_SYS."
