File: SchedaH616/progetto-kicad/pmic.kicad_sch (KiCad schematic)
At the start: 96 parts, among them U201 RK809-5, U202 TCS4525_WT, U203 TPS563201DDCR, U204 AP2112K-1.8TRG1, U205 AP2112K-2.5TRG1, Y201 32.768kHz

Commit message: SchedaH616: passivi 0603, microSD sul bottom, USB-C affiancate
- passivi 0603 di default; 0201/0402 solo per il disaccoppiamento sotto RK3568 e DDR4,
  le serie RGMII/clock/USB, DDR_RZQ, ZQ e VREF della DDR4
  (C: 29x0201, 31x0402, 133x0603; R: 24x0402, 133x0603)
- microSD J401 sul bottom, apertura sul bordo sinistro
- USB-C host J801 e OTG/alimentazione J104 affiancate sul bordo basso, con ESD,
  TPS2553, TPS2121, FUSB302B e SY6280 accanto
- 387 componenti sul top, 52 sul bottom; ERC 0, parita' 0, DRC 0 (solo collegamenti)

Co-Authored-By: Claude Opus 5.5 (1M context) <noreply@anthropic.com>
Parts:
- C205, C206, C207, C208, C210, C214, C217, C222, C225, C226, C227, C228, C229, C230, C231, C232, C233, C234, C236, C237, C238, C239, C240, C241, C242, C243, C244, C247, C248, C254, C255, C258, C259, C260, C261, C262, C263, C264: footprint Capacitor_SMD:C_0402_1005Metric -> Capacitor_SMD:C_0603_1608Metric
- R201, R202, R203, R204, R205, R206, R207, R208, R209, R210, R211, R212, R213, R214, R215, R216, R217: footprint Resistor_SMD:R_0402_1005Metric -> Resistor_SMD:R_0603_1608Metric
