File: SchedaH616/progetto-kicad/radio.kicad_sch (KiCad schematic)
At the start: 17 parts, among them J601 U.FL, U601 AP6256

Commit message: SchedaH616: RK3568 + RK809-5 + TCS4525 + DDR4, placement 50x70
- SoC Allwinner H616 -> Rockchip RK3568 (FCBGA636L, LCSC C2938930): ball map dal pinout
  Rockchip V1.1, verificata sulla tabella 2-1 del datasheet V1.2 (636/636); footprint
  generato (gen_fp.py), confrontato con EasyEDA C2938930
- PMIC AXP313A -> RK809-5 (C2939628) come Rockchip AIoT REF V1.1 / ROCK 3A; TCS4525 per
  VDD_CPU su I2C0 (0x1C); BUCK4 su VDD_NPU (sull'RK809-5 parte spento: non puo' fare il 3.3 V)
- LPDDR4 -> DDR4 x16 K4AAG165WA-BCWE (C2920140) sul canale A, point-to-point, niente VTT,
  VPP da AP2112K-2.5, ZQ 240R, DDR_RZQ del SoC 120R (Hardware Design Guide)
- eMMC su EMMC 8 bit (VCCIO2 1.8 V), microSD su SDMMC0, AP6256 su SDMMC2 + UART8,
  RTL8211F su GMAC0 RGMII (22R TX al SoC e RX al PHY), console UART2_M0, USB-C su OTG0
- Recovery su SARADC_VIN0, reset sulla rete RESETn; TCA6416A tolto
- Bus MIKILAB: BUS_POWER su SPI3_M1, MAIN su SPI2_M1 (CS del DAC su cs-gpios)
- progetto rinominato SchedaRK3568, libreria di progetto Scheda; script portabili Linux/macOS
- ERC 0, parita' 0, DRC 0 (solo collegamenti da fare); placement 439/439

Co-Authored-By: Claude Opus 5.5 (1M context) <noreply@anthropic.com>
Parts:
- removed U601: AP6256, H616:AP6256_LGA-47_12x12mm, symbol H616:AP6256
- added R609: 22R, Resistor_SMD:R_0402_1005Metric, symbol Device:R
- added U601: AP6256, Scheda:AP6256_LGA-47_12x12mm, symbol Scheda:AP6256
Connections:
- net VCC-IO is gone; now on net VCC_3V3: C604.1, C605.1, R603.1, R604.1, R605.1, R606.1, R607.1
- net BT_HOST_WAKE: now also U601.7 (BT_HOST_WAKE)
- net BT_REG_ON: now also U601.34 (BT_REG_ON)
- net BT_UART_CTS: now also U601.41 (UART_RTS_N)
- net BT_UART_RTS: now also U601.44 (UART_CTS_N)
- net BT_UART_RX: now also U601.42 (UART_TXD)
- net BT_UART_TX: now also U601.43 (UART_RXD)
- net BT_WAKE: now also U601.6 (BT_WAKE)
- net GND_D: now also U601.1 (GND), U601.20 (GND), U601.29 (SDIO_VSEL), U601.3 (GND), U601.31 (GND), U601.33 (GND), U601.36 (GND)
- net WL_ANT: now also U601.2 (WL_BT_ANT)
- net WL_HOST_WAKE: now also U601.13 (WL_HOST_WAKE)
- net WL_LDO_OUT: now also U601.21 (VIN_LDO_OUT)
- net WL_REG_ON: now also U601.12 (WL_REG_ON)
- net WL_SDIO_CLK: now also R609.2, U601.17 (SDIO_DATA_CLK)
- net WL_SDIO_CMD: now also U601.16 (SDIO_DATA_CMD)
- net WL_SDIO_D0: now also U601.18 (SDIO_DATA_0)
- net WL_SDIO_D1: now also U601.19 (SDIO_DATA_1)
- net WL_SDIO_D2: now also U601.14 (SDIO_DATA_2)
- net WL_SDIO_D3: now also U601.15 (SDIO_DATA_3)
- net 3V3_PERI renamed VCC_3V3
- net VCC_3V3: now also U601.22 (VDDIO), U601.23 (VIN_LDO), U601.9 (VBAT)
- new net CLK32K: U601.24 (LPO)
- new net WL_SDIO_CLK_S: R609.1
Other:
- note added: "RADIO: AMPAK AP6256 (Wi-Fi 5 + BT 5.0) su SDMMC2_M0 (SDIO, VCCIO6), HCI su UART8_M0 con RTS/CTS (VCCIO4), REG_ON e wake su GPIO. Serie 6xx. Net WL_*/BT_*/CLK32K globali."
- note added: "REG_ON con 100k a GND (radio spenta finche Linux non la accende: GPIO3_D4/D5). Pull-up 10k su CMD e DAT0-3 a VCC_3V3. CLK 22R serie vicino al SoC."
- note added: "UART incrociata: TXD del modulo -> BT_UART_RX (UART8_RX, GPIO2_C6), RXD <- BT_UART_TX (GPIO2_C5), RTS_N -> BT_UART_CTS (GPIO2_B2), CTS_N <- BT_UART_RTS (GPIO2_B1)."
- note added: "VDDIO = VCC_3V3 3.3 V (= VCCIO6/VCCIO4), SDIO 2.0 fino a 50 MHz. VBAT e VIN_LDO da VCC_3V3. LPO 32.768 kHz da CLK32K dell'RK809-5 (quarzo Y201)."
- note removed: "RADIO: AMPAK AP6256 (Wi-Fi 5 + BT 5.0) su SMHC1 PG0-PG5 (SDIO), UART1 PG6-PG9 con RTS/CTS, REG_ON e wake sull'espansore TCA6416A. Serie 6xx. Net WL_*/BT_*/WIFI_32K globali."
- note removed: "REG_ON con 100k a GND (radio spenta finche Linux non la accende dall'espansore). Pull-up 10k su CMD e DAT0-3 a VCC-IO."
- note removed: "UART incrociata: TXD del modulo -> BT_UART_RX (PG7), RXD <- BT_UART_TX (PG6), RTS_N -> BT_UART_CTS (PG9), CTS_N <- BT_UART_RTS (PG8)."
- note removed: "VDDIO = VCC-IO 3.3 V (= VCC_PG), SDIO 2.0 fino a 50 MHz. VBAT e VIN_LDO da 3V3_PERI. LPO 32.768 kHz da X32KFOUT (PG10), derivato dal 24 MHz: da verificare."

Commit message: SchedaH616: componenti specifici dalla libreria MIKILAB
- simbolo e footprint MIKILAB per RK809-5, TCS4525, K4AAG165WA-BCWE, FEMDNN064G-C9A61,
  AP2112K-1.8TRG1, TPS56637RPAR, TPS2121RUXR, SY6280AAC, TPS563201DDCR, TPS2553DBVR,
  TYPE-C-31-M-12, FH12-30S-0.5SH, FPC-05F-28PH20, HR911130C, 25AA02E48T-I/OT, DM3AT-SF-PEJM5;
  simbolo MIKILAB per l'AP6256
- restano nella libreria di progetto: RK3568 (pad EasyEDA da 0.35 mm, niente fanout 5/5 mil),
  simbolo RTL8211F (quello MIKILAB ha pin di alimentazione nascosti), footprint AP6256 LGA-47,
  portapila BS-12; motivazioni in docs/scelte-progetto.md
- kilib.mik() carica simboli e footprint dalla libreria (variabile MIKILAB); matrice ERC:
  pin unspecified dei simboli EasyEDA OK
- netlist identica a 4ca35fc (439 componenti, 314 net); ERC 0, parita' 0, DRC 0 (solo
  collegamenti da fare); footprint corretti nella libreria MIKILAB 8b990c4

Co-Authored-By: Claude Opus 5.5 (1M context) <noreply@anthropic.com>
Parts:
- removed U601: AP6256, Scheda:AP6256_LGA-47_12x12mm, symbol Scheda:AP6256
- added U601: AP6256, Scheda:AP6256_LGA-47_12x12mm, symbol MIKILAB_AP6212:AP6256
Connections:
- net BT_HOST_WAKE: now also U601.7 (BT_HOST_WAKE)
- net BT_REG_ON: now also U601.34 (BT_REG_ON)
- net BT_UART_CTS: now also U601.41 (UART_RTS_N)
- net BT_UART_RTS: now also U601.44 (UART_CTS_N)
- net BT_UART_RX: now also U601.42 (UART_TXD)
- net BT_UART_TX: now also U601.43 (UART_RXD)
- net BT_WAKE: now also U601.6 (BT_WAKE)
- net CLK32K: now also U601.24 (LPO)
- net GND_D: now also U601.1 (GND), U601.20 (GND), U601.29 (SDIO_VSEL), U601.3 (GND), U601.31 (GND), U601.33 (GND), U601.36 (GND)
- net VCC_3V3: now also U601.22 (VDDIO), U601.23 (VIN_LDO), U601.9 (VBAT)
- net WL_ANT: now also U601.2 (WL_BT_ANT)
- net WL_HOST_WAKE: now also U601.13 (WL_HOST_WAKE)
- net WL_LDO_OUT: now also U601.21 (VIN_LDO_OUT)
- net WL_REG_ON: now also U601.12 (WL_REG_ON)
- net WL_SDIO_CLK: now also U601.17 (SDIO_DATA_CLK)
- net WL_SDIO_CMD: now also U601.16 (SDIO_DATA_CMD)
- net WL_SDIO_D0: now also U601.18 (SDIO_DATA_0)
- net WL_SDIO_D1: now also U601.19 (SDIO_DATA_1)
- net WL_SDIO_D2: now also U601.14 (SDIO_DATA_2)
- net WL_SDIO_D3: now also U601.15 (SDIO_DATA_3)
