File: SchedaH616/progetto-kicad/radio.kicad_sch (KiCad schematic)
At the start: 18 parts, among them J601 U.FL, U601 AP6256

Commit message: SchedaH616: passivi 0603, microSD sul bottom, USB-C affiancate
- passivi 0603 di default; 0201/0402 solo per il disaccoppiamento sotto RK3568 e DDR4,
  le serie RGMII/clock/USB, DDR_RZQ, ZQ e VREF della DDR4
  (C: 29x0201, 31x0402, 133x0603; R: 24x0402, 133x0603)
- microSD J401 sul bottom, apertura sul bordo sinistro
- USB-C host J801 e OTG/alimentazione J104 affiancate sul bordo basso, con ESD,
  TPS2553, TPS2121, FUSB302B e SY6280 accanto
- 387 componenti sul top, 52 sul bottom; ERC 0, parita' 0, DRC 0 (solo collegamenti)

Co-Authored-By: Claude Opus 5.5 (1M context) <noreply@anthropic.com>
Parts:
- C602, C604, C605, C606, C607: footprint Capacitor_SMD:C_0402_1005Metric -> Capacitor_SMD:C_0603_1608Metric
- R601, R602, R603, R604, R605, R606, R607, R608: footprint Resistor_SMD:R_0402_1005Metric -> Resistor_SMD:R_0603_1608Metric
