File: SchedaH616/progetto-kicad/alimentazione.kicad_sch (KiCad schematic)
At the start: 62 parts, among them J103 DC-005-5A-2.0, J104 TYPE-C-31-M-12, U101 TPS56637RPAR, U103 TPS2121RUXR, U104 FUSB302BMPX, U105 SY6280AAC, U107 TPD2EUSB30ADRTR, U108 TPS2121RUXR

Commit message: SchedaH616: passivi 0603, microSD sul bottom, USB-C affiancate
- passivi 0603 di default; 0201/0402 solo per il disaccoppiamento sotto RK3568 e DDR4,
  le serie RGMII/clock/USB, DDR_RZQ, ZQ e VREF della DDR4
  (C: 29x0201, 31x0402, 133x0603; R: 24x0402, 133x0603)
- microSD J401 sul bottom, apertura sul bordo sinistro
- USB-C host J801 e OTG/alimentazione J104 affiancate sul bordo basso, con ESD,
  TPS2553, TPS2121, FUSB302B e SY6280 accanto
- 387 componenti sul top, 52 sul bottom; ERC 0, parita' 0, DRC 0 (solo collegamenti)

Co-Authored-By: Claude Opus 5.5 (1M context) <noreply@anthropic.com>
Parts:
- C103, C108, C109, C110, C111, C112, C114, C125, C126, C132, C133, C134, C136: footprint Capacitor_SMD:C_0402_1005Metric -> Capacitor_SMD:C_0603_1608Metric
- R101, R102, R103, R104, R105, R106, R107, R108, R109, R110, R111, R112, R113, R114, R115, R116, R121, R122, R123, R124, R125, R126, R127, R128, R129, R130: footprint Resistor_SMD:R_0402_1005Metric -> Resistor_SMD:R_0603_1608Metric
