File: SchedaH616/progetto-kicad/memorie.kicad_sch (KiCad schematic)
At the start: 54 parts, among them J401 DM3AT-SF-PEJM5, U401 K4AAG165WA-BCWE, U402 FEMDNN064G-C9A61, U403 TPD4E05U06DQA, U404 TPD4E05U06DQA

Commit message: SchedaH616: passivi 0603, microSD sul bottom, USB-C affiancate
- passivi 0603 di default; 0201/0402 solo per il disaccoppiamento sotto RK3568 e DDR4,
  le serie RGMII/clock/USB, DDR_RZQ, ZQ e VREF della DDR4
  (C: 29x0201, 31x0402, 133x0603; R: 24x0402, 133x0603)
- microSD J401 sul bottom, apertura sul bordo sinistro
- USB-C host J801 e OTG/alimentazione J104 affiancate sul bordo basso, con ESD,
  TPS2553, TPS2121, FUSB302B e SY6280 accanto
- 387 componenti sul top, 52 sul bottom; ERC 0, parita' 0, DRC 0 (solo collegamenti)

Co-Authored-By: Claude Opus 5.5 (1M context) <noreply@anthropic.com>
Parts:
- C401, C419, C420, C421, C422, C423, C424, C425, C427: footprint Capacitor_SMD:C_0402_1005Metric -> Capacitor_SMD:C_0603_1608Metric
- R406, R407, R408, R409, R410, R411, R412, R413, R414, R415, R417, R418, R419, R420, R421, R422: footprint Resistor_SMD:R_0402_1005Metric -> Resistor_SMD:R_0603_1608Metric
