File: SchedaH616/progetto-kicad/rete.kicad_sch (KiCad schematic)
At the start: 49 parts, among them J501 HR911130C, U501 RTL8211F-CG, U502 25AA02E48T-I/OT, Y501 25MHz

Commit message: SchedaH616: passivi 0603, microSD sul bottom, USB-C affiancate
- passivi 0603 di default; 0201/0402 solo per il disaccoppiamento sotto RK3568 e DDR4,
  le serie RGMII/clock/USB, DDR_RZQ, ZQ e VREF della DDR4
  (C: 29x0201, 31x0402, 133x0603; R: 24x0402, 133x0603)
- microSD J401 sul bottom, apertura sul bordo sinistro
- USB-C host J801 e OTG/alimentazione J104 affiancate sul bordo basso, con ESD,
  TPS2553, TPS2121, FUSB302B e SY6280 accanto
- 387 componenti sul top, 52 sul bottom; ERC 0, parita' 0, DRC 0 (solo collegamenti)

Co-Authored-By: Claude Opus 5.5 (1M context) <noreply@anthropic.com>
Parts:
- C501, C502, C503, C505, C506, C507, C508, C510, C511, C512, C513, C514, C515: footprint Capacitor_SMD:C_0402_1005Metric -> Capacitor_SMD:C_0603_1608Metric
- R507, R508, R509, R510, R511, R512, R513, R514, R515, R516, R517, R518, R519, R520, R521, R522, R523: footprint Resistor_SMD:R_0402_1005Metric -> Resistor_SMD:R_0603_1608Metric
